File: src/CE_Dongle_V3/CE_Dongle_V3.kicad_sch (KiCad schematic)
At the start: 2 parts, among them J2 8P8C_LED_Shielded

Commit message: layout finished
Parts:
- added G1: 7Sigma Logo, 7Sigma:7Sigma_Logo, symbol Mechanical_7S:7Sigma_Logo
- added G2: Hammond_1551RFLGY, 7Sigma:HAMMOND_1551RFLGY, symbol Mechanical_7S:Hammond_1551RFLGY
- added H1, H2: MH_2.5mm_4mm_OD, 7Sigma:MountingHole_2.5mm_Pad_4mm, symbol Mechanical_7S:MH_2.5mm_4mm_OD
Connections:
- net GND: now also H1.1, H2.1

Commit message: schematic update before production
Connections:
- no-connect marks 0 -> 2
Changed lines of the file:
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@@
 	(generator_version "9.0")
 	(paper "A4")
+	(no_connect
+		(at 30.48 66.04)
+	)
+	(no_connect
+		(at 30.48 68.58)
+	)
 	(wire
 		(pts
@@
 				)
 				(hide yes)
+			)
+		)
+		(property "Manufacturer" ""
+			(at 158.75 173.99 0)
+			(effects
+				(font
+					(size 1 1)
+				)
+				(hide yes)
+			)
+		)
+		(property "Manufacturer Part Number" ""
+			(at 158.75 173.99 0)
+			(effects
+				(font
+					(size 1 1)
+				)
+				(hide yes)
