File: src/CE_Dongle_V3/MUX.kicad_sch (KiCad schematic)
At the start: 24 parts, among them U10 TMUX1208QRSVRQ1, U5 PCF8574RGTR(UMW), U6 PCF8574RGTR(UMW), U7 TMUX1208QRSVRQ1, U8 TMUX1208QRSVRQ1, U9 TMUX1208QRSVRQ1

Commit message: layout finished
Parts:
- removed R31, R32, R33, R34, R35, R36, R6, R7: 10R, 7Sigma:R_0402_1005Metric, symbol Resistor:0402WGF100JTCE
- added C18, C33, C34, C35, C36, C37, C38, C39: 100pF, 7Sigma:C_0402_1005Metric, symbol Capacitor:CC0402JRNPO9BN101
Connections:
- net MUX_IN_1 is gone; now on net IN_1: U10.2 (S1), U7.2 (S1), U8.2 (S1), U9.2 (S1)
- net MUX_IN_2 is gone; now on net IN_2: U10.3 (S2), U7.3 (S2), U8.3 (S2), U9.3 (S2)
- net MUX_IN_3 is gone; now on net IN_3: U10.4 (S3), U7.4 (S3), U8.4 (S3), U9.4 (S3)
- net MUX_IN_4 is gone; now on net IN_4: U10.5 (S4), U7.5 (S4), U8.5 (S4), U9.5 (S4)
- net MUX_IN_5 is gone; now on net IN_5: U10.10 (S5), U7.10 (S5), U8.10 (S5), U9.10 (S5)
- net MUX_IN_6 is gone; now on net IN_6: U10.9 (S6), U7.9 (S6), U8.9 (S6), U9.9 (S6)
- net MUX_IN_7 is gone; now on net IN_7: U10.8 (S7), U7.8 (S7), U8.8 (S7), U9.8 (S7)
- net MUX_IN_8 is gone; now on net IN_8: U10.7 (S8), U7.7 (S8), U8.7 (S8), U9.7 (S8)
- net GND: now also C18.2, C33.2, C34.2, C35.2, C36.1, C37.1, C38.1, C39.1
- net IN_1: now also C39.2
- net IN_2: now also C38.2
- net IN_3: now also C37.2
- net IN_4: now also C36.2
- net IN_5: now also C18.1
- net IN_6: now also C33.1
- net IN_7: now also C34.1
- net IN_8: now also C35.1
