File: src/CE_Dongle_V3/PWR.kicad_sch (KiCad schematic)
At the start: 31 parts, among them J1 USB_C_Receptacle_USB2.0_16P, J5 Conn_01x02, Q1 AO3401A, Q2 AO3401A, Q3 BC817-40-7-F, Q4 BC817-40-7-F, Q5 BC817-40-7-F, U11 TPS70950DBVR, U4 TPS54302DDCR

Commit message: layout finished
Parts:
- added J6: WJ15EDGK-3.81-2P, 7Sigma:TerminalBlock_Plug_Invisible, symbol Connectors:WJ15EDGK-3.81-2P
- R10, R11: Footprint_Name 258 -> 0402

Commit message: schematic update before production
Parts:
- Q1, Q2: comp_type (none) -> PMOS
- Q3, Q4, Q5: comp_type (none) -> NPN
Changed lines of the file:
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@@
 		)
 		(property "Value" "BC817-40-7-F"
-			(at 119.38 102.87 90)
+			(at 119.38 102.87 0)
 			(effects
 				(font
@@
 			)
 		)
+		(property "comp_type" "NPN"
+			(at 114.3 93.98 0)
+			(effects
+				(font
+					(size 1 1)
+				)
+				(hide yes)
+			)
+		)
 		(pin "1"
 		)
@@
 		)
 		(property "Value" "BC817-40-7-F"
-			(at 132.08 59.69 90)
+			(at 132.08 59.69 0)
 			(effects
 				(font
@@
 			)
 		)
+		(property "comp_type" "NPN"
+			(at 127 50.8 0)
+			(effects
+				(font
+					(size 1 1)
+				)
+				(hide yes)
+			)
+		)
 		(pin "1"
 		)
@@
 		)
 		(property "Value" "AO3401A"
-			(at 133.858 68.072 90)
+			(at 133.858 68.072 0)
 			(effects
 				(font
@@
 			)
 		)
+		(property "comp_type" "PMOS"
+			(at 129.54 73.66 0)
+			(effects
+				(font
+					(size 1 1)
+				)
+				(hide yes)
+			)
+		)
 		(pin "1"
 		)
@@
 		)
 		(property "Value" "AO3401A"
-			(at 133.858 32.512 90)
+			(at 133.858 32.512 0)
 			(effects
 				(font
@@
 			)
 		)
+		(property "comp_type" "PMOS"
+			(at 129.54 38.1 0)
+			(effects
+				(font
+					(size 1 1)
+				)
+				(hide yes)
+			)
+		)
 		(pin "1"
 		)
@@
 		)
 		(property "Value" "BC817-40-7-F"
-			(at 132.08 97.79 90)
+			(at 132.08 97.79 0)
 			(effects
 				(font
@@
 			)
 		)
+		(property "comp_type" "NPN"
+			(at 127 88.9 0)
+			(effects
+				(font
+					(size 1 1)
+				)
+				(hide yes)
+			)
+		)
 		(pin "1"
 		)
@@
 			)
 		)
-		(property "Datasheet" "https://atta.szlcsc.com/upload/public/pdf/source/20200306/C422600_1E6D84923E4A46A82E41ADD87F860B5C.pdf"
+		(property "Datasheet" "https://lcsc.com/product-detail/Chip-Resistor-Surface-Mount-UniOhm_5-1KR-5101-1_C25905.html"
 			(at 53.34 76.2 0)
 			(effects
@@
 		(exclude_from_sim no)
 		(in_bom yes)
-		(on_board yes)
+		(on_board no)
 		(dnp no)
 		(property "Reference" "J6"
@@
 			)
 		)
-		(property "Datasheet" "https://atta.szlcsc.com/upload/public/pdf/source/20200306/C422600_1E6D84923E4A46A82E41ADD87F860B5C.pdf"
+		(property "Datasheet" "https://lcsc.com/product-detail/Chip-Resistor-Surface-Mount-UniOhm_5-1KR-5101-1_C25905.html"
 			(at 59.69 78.74 0)
 			(effects
