File: src/EG915U.kicad_sch (KiCad schematic)
At the start: 23 parts, among them U13 EG915U

Commit message: ongoing work
Connections:
- net +3V3 is gone; now on net 3V8: C63.1, C78.1, C79.1
- net 3V8: now reaches U13.32 (VBAT_BB)
- net 3V8: now also U13.33 (VBAT_BB), U13.52 (VBAT_RF), U13.53 (VBAT_RF)
- net GNDD renamed GND
