File: src/EG915U.kicad_sch (KiCad schematic)
At the start: 23 parts, among them U13 EG915U

Commit message: layout + lib swap to http library. changed up the 10u and 47u caps for cheaper alternative
Parts:
- C63, C75: symbol Capacitor:CL05B104KO5NNNC -> 7Sigma:CL05B104KO5NNNC
- C64, C65, C74: symbol Capacitor:GRM155R61H105KE05D -> 7Sigma:GRM155R61H105KE05D
- C66, C67: symbol Capacitor:GJM1555C1H1R2WB01D -> 7Sigma:GJM1555C1H1R2WB01D
- C68, C69, C70, C71, C72, C73: symbol Capacitor:CC0402JRNPO9BN330 -> 7Sigma:CC0402JRNPO9BN330
- C78, C79: symbol Capacitor:CS3225X7R476K160NRL -> 7Sigma:CS3225X7R476K160NRL
- R46: symbol Resistor:0402WGF0000TCE -> 7Sigma:0402WGF0000TCE
- TP10, TP11, TP12, TP7, TP8, TP9: symbol TestPoints:TestPoint_Pad_D1.5mm -> 7Sigma:TestPoint_Pad_D1.5mm
- U13: symbol ICs:EG915UEUAC-N05-SNNSA -> 7Sigma:EG915UEUAC-N05-SNNSA
Changed lines of the file:
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@@
 	)
 	(symbol
-		(lib_id "Capacitor:CC0402JRNPO9BN330")
+		(lib_id "7Sigma:CC0402JRNPO9BN330")
 		(at 152.4 143.51 0)
 		(unit 1)
@@
 	)
 	(symbol
-		(lib_id "Resistor:0402WGF0000TCE")
+		(lib_id "7Sigma:0402WGF0000TCE")
 		(at 151.13 50.8 270)
 		(mirror x)
@@
 	)
 	(symbol
-		(lib_id "Capacitor:GRM155R61H105KE05D")
+		(lib_id "7Sigma:GRM155R61H105KE05D")
 		(at 26.67 107.95 0)
 		(unit 1)
@@
 	)
 	(symbol
-		(lib_id "Capacitor:CL05B104KO5NNNC")
+		(lib_id "7Sigma:CL05B104KO5NNNC")
 		(at 34.29 107.95 0)
 		(unit 1)
@@
 	)
 	(symbol
-		(lib_id "TestPoints:TestPoint_Pad_D1.5mm")
+		(lib_id "7Sigma:TestPoint_Pad_D1.5mm")
 		(at 180.34 60.96 90)
 		(mirror x)
@@
 	)
 	(symbol
-		(lib_id "ICs:EG915UEUAC-N05-SNNSA")
+		(lib_id "7Sigma:EG915UEUAC-N05-SNNSA")
 		(at 198.12 33.02 0)
 		(unit 4)
@@
 	)
 	(symbol
-		(lib_id "TestPoints:TestPoint_Pad_D1.5mm")
+		(lib_id "7Sigma:TestPoint_Pad_D1.5mm")
 		(at 180.34 66.04 90)
 		(mirror x)
@@
 	)
 	(symbol
-		(lib_id "Capacitor:GRM155R61H105KE05D")
+		(lib_id "7Sigma:GRM155R61H105KE05D")
 		(at 102.87 29.21 0)
 		(unit 1)
@@
 	)
 	(symbol
-		(lib_id "ICs:EG915UEUAC-N05-SNNSA")
+		(lib_id "7Sigma:EG915UEUAC-N05-SNNSA")
 		(at 76.2 96.52 0)
 		(unit 3)
@@
 	)
 	(symbol
-		(lib_id "Capacitor:CC0402JRNPO9BN330")
+		(lib_id "7Sigma:CC0402JRNPO9BN330")
 		(at 137.16 143.51 0)
 		(unit 1)
@@
 	)
 	(symbol
-		(lib_id "Capacitor:CL05B104KO5NNNC")
+		(lib_id "7Sigma:CL05B104KO5NNNC")
 		(at 40.64 29.21 0)
 		(unit 1)
@@
 	)
 	(symbol
-		(lib_id "TestPoints:TestPoint_Pad_D1.5mm")
+		(lib_id "7Sigma:TestPoint_Pad_D1.5mm")
 		(at 180.34 96.52 90)
 		(mirror x)
@@
 	)
 	(symbol
-		(lib_id "Capacitor:CC0402JRNPO9BN330")
+		(lib_id "7Sigma:CC0402JRNPO9BN330")
 		(at 167.64 143.51 0)
 		(unit 1)
@@
 	)
 	(symbol
-		(lib_id "TestPoints:TestPoint_Pad_D1.5mm")
+		(lib_id "7Sigma:TestPoint_Pad_D1.5mm")
 		(at 180.34 63.5 90)
 		(mirror x)
@@
 	)
 	(symbol
-		(lib_id "Capacitor:GJM1555C1H1R2WB01D")
+		(lib_id "7Sigma:GJM1555C1H1R2WB01D")
 		(at 160.02 54.61 0)
 		(unit 1)
@@
 	)
 	(symbol
-		(lib_id "TestPoints:TestPoint_Pad_D1.5mm")
+		(lib_id "7Sigma:TestPoint_Pad_D1.5mm")
 		(at 180.34 99.06 90)
 		(mirror x)
@@
 	)
 	(symbol
-		(lib_id "Capacitor:CC0402JRNPO9BN330")
+		(lib_id "7Sigma:CC0402JRNPO9BN330")
 		(at 160.02 143.51 0)
 		(unit 1)
@@
 	)
 	(symbol
-		(lib_id "ICs:EG915UEUAC-N05-SNNSA")
+		(lib_id "7Sigma:EG915UEUAC-N05-SNNSA")
 		(at 198.12 78.74 0)
 		(unit 2)
@@
 	)
 	(symbol
-		(lib_id "Capacitor:CC0402JRNPO9BN330")
+		(lib_id "7Sigma:CC0402JRNPO9BN330")
 		(at 144.78 143.51 0)
 		(unit 1)
@@
 	)
 	(symbol
-		(lib_id "Capacitor:CS3225X7R476K160NRL")
+		(lib_id "7Sigma:CS3225X7R476K160NRL")
 		(at 25.4 29.21 0)
 		(unit 1)
@@
 	)
 	(symbol
-		(lib_id "Capacitor:GJM1555C1H1R2WB01D")
+		(lib_id "7Sigma:GJM1555C1H1R2WB01D")
 		(at 139.7 54.61 0)
 		(unit 1)
@@
 	)
 	(symbol
-		(lib_id "ICs:EG915UEUAC-N05-SNNSA")
+		(lib_id "7Sigma:EG915UEUAC-N05-SNNSA")
 		(at 76.2 50.8 0)
 		(unit 1)
@@
 	)
 	(symbol
-		(lib_id "Capacitor:CS3225X7R476K160NRL")
+		(lib_id "7Sigma:CS3225X7R476K160NRL")
 		(at 33.02 29.21 0)
 		(unit 1)
@@
 	)
 	(symbol
-		(lib_id "TestPoints:TestPoint_Pad_D1.5mm")
+		(lib_id "7Sigma:TestPoint_Pad_D1.5mm")
 		(at 180.34 58.42 90)
 		(mirror x)
@@
 	)
 	(symbol
-		(lib_id "ICs:EG915UEUAC-N05-SNNSA")
+		(lib_id "7Sigma:EG915UEUAC-N05-SNNSA")
 		(at 76.2 139.7 0)
 		(unit 5)
@@
 	)
 	(symbol
-		(lib_id "Capacitor:CC0402JRNPO9BN330")
+		(lib_id "7Sigma:CC0402JRNPO9BN330")
 		(at 175.26 143.51 0)
 		(unit 1)
@@
 	)
 	(symbol
-		(lib_id "Capacitor:GRM155R61H105KE05D")
+		(lib_id "7Sigma:GRM155R61H105KE05D")
 		(at 110.49 29.21 0)
 		(unit 1)
