File: src/LE310X1.kicad_sch (KiCad schematic)
At the start: 19 parts, among them U12 LE310X1

Commit message: ongoing work
Connections:
- net +3V3 renamed 3V8
- net GNDD renamed GND
Changed lines of the file:
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@@
 	)
 	(symbol
-		(lib_id "power:GNDD")
+		(lib_id "Power:GND")
 		(at 27.94 45.72 0)
 		(unit 1)
@@
 			)
 		)
-		(property "Value" "GNDD"
+		(property "Value" "GND"
 			(at 27.94 48.895 0)
 			(show_name no)
@@
 			)
 		)
-		(property "Description" "Power symbol creates a global label with name \"GNDD\" , digital ground"
+		(property "Description" "Power symbol creates a global label with name \"GND\", digital ground"
 			(at 27.94 45.72 0)
 			(hide yes)
@@
 	)
 	(symbol
-		(lib_id "power:GNDD")
+		(lib_id "Power:GND")
 		(at 50.8 45.72 0)
 		(unit 1)
@@
 			)
 		)
-		(property "Value" "GNDD"
+		(property "Value" "GND"
 			(at 50.8 48.895 0)
 			(show_name no)
@@
 			)
 		)
-		(property "Description" "Power symbol creates a global label with name \"GNDD\" , digital ground"
+		(property "Description" "Power symbol creates a global label with name \"GND\", digital ground"
 			(at 50.8 45.72 0)
 			(hide yes)
@@
 	)
 	(symbol
-		(lib_id "power:GNDD")
+		(lib_id "Power:GND")
 		(at 38.1 124.46 0)
 		(unit 1)
@@
 			)
 		)
-		(property "Value" "GNDD"
+		(property "Value" "GND"
 			(at 38.1 127.635 0)
 			(show_name no)
@@
 			)
 		)
-		(property "Description" "Power symbol creates a global label with name \"GNDD\" , digital ground"
+		(property "Description" "Power symbol creates a global label with name \"GND\", digital ground"
 			(at 38.1 124.46 0)
 			(hide yes)
@@
 	)
 	(symbol
-		(lib_id "power:GNDD")
+		(lib_id "Power:GND")
 		(at 177.8 33.02 0)
 		(mirror y)
@@
 			)
 		)
-		(property "Value" "GNDD"
+		(property "Value" "GND"
 			(at 177.8 36.195 0)
 			(show_name no)
@@
 			)
 		)
-		(property "Description" "Power symbol creates a global label with name \"GNDD\" , digital ground"
+		(property "Description" "Power symbol creates a global label with name \"GND\", digital ground"
 			(at 177.8 33.02 0)
 			(hide yes)
@@
 	)
 	(symbol
-		(lib_id "power:GNDD")
+		(lib_id "Power:GND")
 		(at 99.06 111.76 270)
 		(unit 1)
@@
 			)
 		)
-		(property "Value" "GNDD"
+		(property "Value" "GND"
 			(at 95.885 111.76 0)
 			(show_name no)
@@
 			)
 		)
-		(property "Description" "Power symbol creates a global label with name \"GNDD\" , digital ground"
+		(property "Description" "Power symbol creates a global label with name \"GND\", digital ground"
 			(at 99.06 111.76 0)
 			(hide yes)
@@
 	)
 	(symbol
-		(lib_id "power:GNDD")
+		(lib_id "Power:GND")
 		(at 35.56 45.72 0)
 		(unit 1)
@@
 			)
 		)
-		(property "Value" "GNDD"
+		(property "Value" "GND"
 			(at 35.56 48.895 0)
 			(show_name no)
@@
 			)
 		)
-		(property "Description" "Power symbol creates a global label with name \"GNDD\" , digital ground"
+		(property "Description" "Power symbol creates a global label with name \"GND\", digital ground"
 			(at 35.56 45.72 0)
 			(hide yes)
@@
 	)
 	(symbol
-		(lib_id "power:GNDD")
+		(lib_id "Power:GND")
 		(at 30.48 124.46 0)
 		(unit 1)
@@
 			)
 		)
-		(property "Value" "GNDD"
+		(property "Value" "GND"
 			(at 30.48 127.635 0)
 			(show_name no)
@@
 			)
 		)
-		(property "Description" "Power symbol creates a global label with name \"GNDD\" , digital ground"
+		(property "Description" "Power symbol creates a global label with name \"GND\", digital ground"
 			(at 30.48 124.46 0)
 			(hide yes)
@@
 	)
 	(symbol
-		(lib_id "power:GNDD")
+		(lib_id "Power:GND")
 		(at 43.18 45.72 0)
 		(unit 1)
@@
 			)
 		)
-		(property "Value" "GNDD"
+		(property "Value" "GND"
 			(at 43.18 48.895 0)
 			(show_name no)
@@
 			)
 		)
-		(property "Description" "Power symbol creates a global label with name \"GNDD\" , digital ground"
+		(property "Description" "Power symbol creates a global label with name \"GND\", digital ground"
 			(at 43.18 45.72 0)
 			(hide yes)
@@
 	)
 	(symbol
-		(lib_id "power:+3V3")
+		(lib_id "Power:3V8")
 		(at 99.06 22.86 0)
 		(unit 1)
@@
 			)
 		)
-		(property "Value" "+3V3"
+		(property "Value" "3V8"
 			(at 99.06 19.304 0)
 			(show_name no)
@@
 			)
 		)
-		(property "Description" "Power symbol creates a global label with name \"+3V3\""
+		(property "Description" "Power symbol creates a global label with name \"3V8\""
 			(at 99.06 22.86 0)
 			(hide yes)
@@
 	)
 	(symbol
-		(lib_id "power:GNDD")
+		(lib_id "Power:GND")
 		(at 76.2 33.02 0)
 		(unit 1)
@@
 			)
 		)
-		(property "Value" "GNDD"
+		(property "Value" "GND"
 			(at 76.2 36.195 0)
 			(show_name no)
@@
 			)
 		)
-		(property "Description" "Power symbol creates a global label with name \"GNDD\" , digital ground"
+		(property "Description" "Power symbol creates a global label with name \"GND\", digital ground"
 			(at 76.2 33.02 0)
 			(hide yes)
@@
 	)
 	(symbol
-		(lib_id "power:GNDD")
+		(lib_id "Power:GND")
 		(at 58.42 45.72 0)
 		(unit 1)
@@
 			)
 		)
-		(property "Value" "GNDD"
+		(property "Value" "GND"
 			(at 58.42 48.895 0)
 			(show_name no)
@@
 			)
 		)
-		(property "Description" "Power symbol creates a global label with name \"GNDD\" , digital ground"
+		(property "Description" "Power symbol creates a global label with name \"GND\", digital ground"
 			(at 58.42 45.72 0)
 			(hide yes)
@@
 	)
 	(symbol
-		(lib_id "power:GNDD")
+		(lib_id "Power:GND")
 		(at 20.32 45.72 0)
 		(unit 1)
@@
 			)
 		)
-		(property "Value" "GNDD"
+		(property "Value" "GND"
 			(at 20.32 48.895 0)
 			(show_name no)
@@
 			)
 		)
-		(property "Description" "Power symbol creates a global label with name \"GNDD\" , digital ground"
+		(property "Description" "Power symbol creates a global label with name \"GND\", digital ground"
 			(at 20.32 45.72 0)
 			(hide yes)
@@
 	)
 	(symbol
-		(lib_id "power:GNDD")
+		(lib_id "Power:GND")
 		(at 83.82 33.02 0)
 		(unit 1)
@@
 			)
 		)
-		(property "Value" "GNDD"
+		(property "Value" "GND"
 			(at 83.82 36.195 0)
 			(show_name no)
@@
 			)
 		)
-		(property "Description" "Power symbol creates a global label with name \"GNDD\" , digital ground"
+		(property "Description" "Power symbol creates a global label with name \"GND\", digital ground"
 			(at 83.82 33.02 0)
 			(hide yes)
@@
 	)
 	(symbol
-		(lib_id "power:GNDD")
+		(lib_id "Power:GND")
 		(at 91.44 33.02 0)
 		(unit 1)
@@
 			)
 		)
-		(property "Value" "GNDD"
+		(property "Value" "GND"
 			(at 91.44 36.195 0)
 			(show_name no)
@@
 			)
 		)
-		(property "Description" "Power symbol creates a global label with name \"GNDD\" , digital ground"
+		(property "Description" "Power symbol creates a global label with name \"GND\", digital ground"
 			(at 91.44 33.02 0)
 			(hide yes)
@@
 	)
 	(symbol
-		(lib_id "power:GNDD")
+		(lib_id "Power:GND")
 		(at 157.48 33.02 0)
 		(mirror y)
@@
 			)
 		)
-		(property "Value" "GNDD"
+		(property "Value" "GND"
 			(at 157.48 36.195 0)
 			(show_name no)
@@
 			)
 		)
-		(property "Description" "Power symbol creates a global label with name \"GNDD\" , digital ground"
+		(property "Description" "Power symbol creates a global label with name \"GND\", digital ground"
 			(at 157.48 33.02 0)
 			(hide yes)
