File: src/LE310X1.kicad_sch (KiCad schematic)
At the start: 19 parts, among them U12 LE310X1

Commit message: layout + lib swap to http library. changed up the 10u and 47u caps for cheaper alternative
Parts:
- C46, C48: symbol Capacitor:CL05B104KO5NNNC -> 7Sigma:CL05B104KO5NNNC
- C49: symbol Capacitor:GRM155R61H105KE05D -> 7Sigma:GRM155R61H105KE05D
- C54, C55: symbol Capacitor:GJM1555C1H1R2WB01D -> 7Sigma:GJM1555C1H1R2WB01D
- C56, C57, C58, C59, C60, C61: symbol Capacitor:CC0402JRNPO9BN330 -> 7Sigma:CC0402JRNPO9BN330
- C76, C77: symbol Capacitor:CS3225X7R476K160NRL -> 7Sigma:CS3225X7R476K160NRL
- R32: symbol Resistor:0402WGF0000TCE -> 7Sigma:0402WGF0000TCE
- TP3, TP4, TP5, TP6: symbol TestPoints:TestPoint_Pad_D1.5mm -> 7Sigma:TestPoint_Pad_D1.5mm
- U12: symbol ICs:LE310X1-EU -> 7Sigma:LE310X1-EU
Changed lines of the file:
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@@
 	)
 	(symbol
-		(lib_id "Capacitor:CL05B104KO5NNNC")
+		(lib_id "7Sigma:CL05B104KO5NNNC")
 		(at 91.44 29.21 0)
 		(unit 1)
@@
 	)
 	(symbol
-		(lib_id "Capacitor:CC0402JRNPO9BN330")
+		(lib_id "7Sigma:CC0402JRNPO9BN330")
 		(at 35.56 41.91 0)
 		(unit 1)
@@
 	)
 	(symbol
-		(lib_id "Capacitor:CS3225X7R476K160NRL")
+		(lib_id "7Sigma:CS3225X7R476K160NRL")
 		(at 76.2 29.21 0)
 		(unit 1)
@@
 	)
 	(symbol
-		(lib_id "Capacitor:CL05B104KO5NNNC")
+		(lib_id "7Sigma:CL05B104KO5NNNC")
 		(at 38.1 120.65 0)
 		(unit 1)
@@
 	)
 	(symbol
-		(lib_id "TestPoints:TestPoint_Pad_D1.5mm")
+		(lib_id "7Sigma:TestPoint_Pad_D1.5mm")
 		(at 137.16 33.02 270)
 		(unit 1)
@@
 	)
 	(symbol
-		(lib_id "Capacitor:GJM1555C1H1R2WB01D")
+		(lib_id "7Sigma:GJM1555C1H1R2WB01D")
 		(at 157.48 29.21 0)
 		(mirror y)
@@
 	)
 	(symbol
-		(lib_id "TestPoints:TestPoint_Pad_D1.5mm")
+		(lib_id "7Sigma:TestPoint_Pad_D1.5mm")
 		(at 157.48 127 270)
 		(unit 1)
@@
 	)
 	(symbol
-		(lib_id "Capacitor:CC0402JRNPO9BN330")
+		(lib_id "7Sigma:CC0402JRNPO9BN330")
 		(at 58.42 41.91 0)
 		(unit 1)
@@
 	)
 	(symbol
-		(lib_id "Capacitor:CS3225X7R476K160NRL")
+		(lib_id "7Sigma:CS3225X7R476K160NRL")
 		(at 83.82 29.21 0)
 		(unit 1)
@@
 	)
 	(symbol
-		(lib_id "Capacitor:GRM155R61H105KE05D")
+		(lib_id "7Sigma:GRM155R61H105KE05D")
 		(at 30.48 120.65 0)
 		(unit 1)
@@
 	)
 	(symbol
-		(lib_id "ICs:LE310X1-EU")
+		(lib_id "7Sigma:LE310X1-EU")
 		(at 119.38 102.87 0)
 		(unit 1)
@@
 	)
 	(symbol
-		(lib_id "Capacitor:GJM1555C1H1R2WB01D")
+		(lib_id "7Sigma:GJM1555C1H1R2WB01D")
 		(at 177.8 29.21 0)
 		(mirror y)
@@
 	)
 	(symbol
-		(lib_id "Capacitor:CC0402JRNPO9BN330")
+		(lib_id "7Sigma:CC0402JRNPO9BN330")
 		(at 27.94 41.91 0)
 		(unit 1)
@@
 	)
 	(symbol
-		(lib_id "Capacitor:CC0402JRNPO9BN330")
+		(lib_id "7Sigma:CC0402JRNPO9BN330")
 		(at 20.32 41.91 0)
 		(unit 1)
@@
 	)
 	(symbol
-		(lib_id "Capacitor:CC0402JRNPO9BN330")
+		(lib_id "7Sigma:CC0402JRNPO9BN330")
 		(at 43.18 41.91 0)
 		(unit 1)
@@
 	)
 	(symbol
-		(lib_id "TestPoints:TestPoint_Pad_D1.5mm")
+		(lib_id "7Sigma:TestPoint_Pad_D1.5mm")
 		(at 137.16 30.48 270)
 		(unit 1)
@@
 	)
 	(symbol
-		(lib_id "Resistor:0402WGF0000TCE")
+		(lib_id "7Sigma:0402WGF0000TCE")
 		(at 166.37 25.4 90)
 		(unit 1)
@@
 	)
 	(symbol
-		(lib_id "TestPoints:TestPoint_Pad_D1.5mm")
+		(lib_id "7Sigma:TestPoint_Pad_D1.5mm")
 		(at 137.16 35.56 270)
 		(unit 1)
@@
 	)
 	(symbol
-		(lib_id "Capacitor:CC0402JRNPO9BN330")
+		(lib_id "7Sigma:CC0402JRNPO9BN330")
 		(at 50.8 41.91 0)
 		(unit 1)
