File: src/CE_Dongle_V3.kicad_pcb (KiCad board)
At the start: 4 copper layers, 52 x 105.2 mm, 193 parts, among them J1 USB_C_Receptacle_USB2.0_16P, J11 Conn_IPEX, J12 Conn_IPEX, J2 Conn_01x02, J3 Conn_01x02, J4 8P8C_LED_Shielded, J5 Conn_01x02, J6 Conn_01x02, J7 Conn_01x02, J9 SIM_NANO_Socket, Q11 SI2308A, Q12 SI2308A, Q13 SI2308A, Q14 SI2308A, Q15 SI2308A, Q18 SI2308A, Q3 AON7264E, Q4 SI2319A, Q5 SI2319A, Q6 AON7264E, Q7 BC817-40-7-F, Q8 BC817-40-7-F, SW1 TS24CA, SW2 TC-6615-9.0-160G, U1 ESP32-C6, U10 TMUX1208RSVR, U11 TPS7B69xx, U14 TPS54302DDCR, U15 TXS0104ERGYR, U16 LE910R1, U17 WS2812, U18 WS2812, U2 SP3485, U20 WS2812, U3 W25Q64JVSSIQ, U4 TPS54302DDCR, U5 PCF8574RGTR(UMW), U6 PCF8574RGTR(UMW), U7 TMUX1208RSVR, U8 TMUX1208RSVR, U9 TMUX1208RSVR, Y1 40MHz

Commit message: pcb layout continued
Parts:
- moved R10 13.6 mm to (122.2, 79.5), turned to 180 degrees
- moved R11 11.5 mm to (122.2, 78.4), turned to 180 degrees
- moved C47 3.60 mm to (148.8, 89.0), turned to 90 degrees
- moved U15 1.80 mm to (122.2, 83.9)
- moved C50 1.80 mm to (123.7, 87.0)
- moved C51 1.80 mm to (120.7, 87.0)
- moved R31 1.10 mm to (117.2, 62.1), turned to 90 degrees
- moved C22 0.58 mm to (137.7, 89.3), turned to 180 degrees
- moved C46 0.30 mm to (130.9, 89.0), turned to 90 degrees
- moved R14 0.20 mm to (118.5, 69.9)
- moved C10 0.10 mm to (123.6, 58.7)
- moved C8 0.10 mm to (121.4, 58.7)
- moved L1 0.10 mm to (122.5, 58.7)
- turned U17 to 90 degrees
- turned U18 to 90 degrees
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Routing:
- net 3V3: track 53.6 -> 230.4 mm, vias 25 -> 29
- net 3V8: track 27.4 -> 123.9 mm, vias 29 -> 32
- net /MCU/O2_CTRL: track 7.45 -> 91.7 mm, vias 0 -> 2
- net /MCU/BUTTON: track 0.00 -> 80.7 mm, vias 0 -> 1
- net /PWR/CON_USB_D+: track 2.74 -> 79.0 mm, vias 0 -> 2
- net /MISC/TEMP: track 0.92 -> 75.4 mm, vias 0 -> 2
- net /PWR/CON_USB_D-: track 2.90 -> 77.1 mm, vias 0 -> 2
- net /MCU/O1_CTRL: track 7.39 -> 81.5 mm, vias 0 -> 4
- net /MCU/I2C_SCL: track 18.5 -> 72.0 mm
- net /MCU/I2C_SDA: track 19.6 -> 67.0 mm
- net /MCU/MODBUS_TX: track 0.00 -> 39.5 mm, vias 0 -> 2
- net /MCU/MODBUS_TX_EN: track 5.38 -> 43.3 mm, vias 0 -> 2
- net /LTE/PWR_MON: track 1.79 -> 38.6 mm, vias 0 -> 2
- net /MCU/MODBUS_RX: track 0.97 -> 37.7 mm, vias 0 -> 2
- net /LTE/UART_RX: track 1.26 -> 35.3 mm, vias 0 -> 2
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- added copper zone on In2.Cu, net 3V8
- added copper zone on In1.Cu, net Net-(U14-SW)
- added copper zone on In1.Cu, net Net-(U4-SW)

Commit message: layout continued
Parts:
- moved C32 0.68 mm to (128.9, 108.2)
- moved C1 0.30 mm to (126.2, 70.4)
- moved C71 0.28 mm to (154.1, 52.1)
- moved R31 0.20 mm to (117.2, 62.3)
- turned D3 to 0 degrees
Connections:
- J11 pad 4: unconnected-(J11-PT-Pad4) -> GND
- J12 pad 4: unconnected-(J12-PT-Pad4) -> GND
Routing:
- net /MCU/RST: track 4.94 -> 99.0 mm, vias 1 -> 4
- net /MISC/VSUPPLY: track 35.7 -> 112.4 mm, vias 10 -> 12
- net 5V0: track 13.8 -> 68.5 mm, vias 8 -> 9
- net /MUX/OUT_B: track 49.6 -> 101.1 mm, vias 3 -> 7
- net /MUX/OUT_A: track 34.7 -> 82.6 mm, vias 3 -> 9
- net /MUX/IN_8: track 43.6 -> 17.9 mm, vias 5 -> 2
- net /MISC/OUT2: track 17.1 -> 40.0 mm
- net /MISC/OUT1: track 13.5 -> 36.1 mm
- net Net-(D9-C): track 4.99 -> 18.3 mm, vias 0 -> 2
- net /MUX/IN_3: track 44.9 -> 53.6 mm
- net /MCU/O1_CTRL: track 81.5 -> 90.0 mm, vias 4 -> 2
- net /LTE/RF_OUT: track 0.00 -> 4.75 mm
- net /MUX/IN_5: track 38.5 -> 33.8 mm
- net GND: track 176.6 -> 181.2 mm, vias 582 -> 556
- net Net-(Q4-G): track 1.20 -> 5.10 mm, vias 0 -> 2
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- added copper zone on In2.Cu, net /MISC/VSUPPLY
- added copper zone on F.Cu, net 5V0
- added copper zone on F.Cu, net Net-(F1-Pad2)
- added copper zone on F.Cu, net Net-(F2-Pad2)

Commit message: layout + lib swap to http library. changed up the 10u and 47u caps for cheaper alternative
Parts:
- added TP1: TestPoint, PCM_7Sigma:TestPoint_Pad_D1.5mm, B.Cu at (158.8, 123.5)
- added TP10: TestPoint, PCM_7Sigma:TestPoint_Pad_D1.5mm, B.Cu at (148.4, 83.4)
- added TP11: TestPoint, PCM_7Sigma:TestPoint_Pad_D1.5mm, B.Cu at (159.9, 82.9)
- added TP12: TestPoint, PCM_7Sigma:TestPoint_Pad_D1.5mm, B.Cu at (155.4, 63.5)
- added TP13: TestPoint, PCM_7Sigma:TestPoint_Pad_D1.5mm, B.Cu at (159.8, 77.4)
- added TP14: TestPoint, PCM_7Sigma:TestPoint_Pad_D1.5mm, B.Cu at (161.1, 80.0)
- added TP15: TestPoint, PCM_7Sigma:TestPoint_Pad_D1.5mm, B.Cu at (163.1, 83.9)
- added TP16: TestPoint, PCM_7Sigma:TestPoint_Pad_D1.5mm, B.Cu at (135.2, 75.2)
- added TP17: TestPoint, PCM_7Sigma:TestPoint_Pad_D1.5mm, B.Cu at (143.5, 79.9)
- added TP18: TestPoint, PCM_7Sigma:TestPoint_Pad_D1.5mm, B.Cu at (157.3, 82.1)
- added TP19: TestPoint, PCM_7Sigma:TestPoint_Pad_D1.5mm, B.Cu at (160.2, 89.5)
- added TP2: TestPoint, PCM_7Sigma:TestPoint_Pad_D1.5mm, B.Cu at (158.4, 127.0)
- added TP20: TestPoint, PCM_7Sigma:TestPoint_Pad_D1.5mm, B.Cu at (162.2, 93.7)
- added TP21: TestPoint, PCM_7Sigma:TestPoint_Pad_D1.5mm, B.Cu at (156.8, 97.1)
- added TP22: TestPoint, PCM_7Sigma:TestPoint_Pad_D1.5mm, B.Cu at (160.3, 97.9)
- added TP23: TestPoint, PCM_7Sigma:TestPoint_Pad_D1.5mm, B.Cu at (150.2, 98.7)
- added TP24: TestPoint, PCM_7Sigma:TestPoint_Pad_D1.5mm, B.Cu at (156.5, 67.0)
- added TP25: TestPoint, PCM_7Sigma:TestPoint_Pad_D1.5mm, B.Cu at (128.3, 89.2)
- added TP26: TestPoint, PCM_7Sigma:TestPoint_Pad_D1.5mm, B.Cu at (118.2, 95.3)
- added TP27: TestPoint, PCM_7Sigma:TestPoint_Pad_D1.5mm, B.Cu at (125.6, 76.7)
- added TP28: TestPoint, PCM_7Sigma:TestPoint_Pad_D1.5mm, B.Cu at (118.2, 103.3)
- added TP29: TestPoint, PCM_7Sigma:TestPoint_Pad_D1.5mm, B.Cu at (119.4, 105.9)
- added TP30: TestPoint, PCM_7Sigma:TestPoint_Pad_D1.5mm, B.Cu at (127.2, 94.7)
- added TP31: TestPoint, PCM_7Sigma:TestPoint_Pad_D1.5mm, B.Cu at (118.4, 58.3)
- added TP33: TestPoint, PCM_7Sigma:TestPoint_Pad_D1.5mm, B.Cu at (136.4, 56.6)
- added TP34: TestPoint, PCM_7Sigma:TestPoint_Pad_D1.5mm, B.Cu at (144.8, 97.3)
- added TP35: TestPoint, PCM_7Sigma:TestPoint_Pad_D1.5mm, B.Cu at (155.7, 122.9)
- added TP36: TestPoint, PCM_7Sigma:TestPoint_Pad_D1.5mm, B.Cu at (162.1, 127.3)
- added TP37: TestPoint, PCM_7Sigma:TestPoint_Pad_D1.5mm, B.Cu at (120.0, 139.8)
- added TP38: TestPoint, PCM_7Sigma:TestPoint_Pad_D1.5mm, B.Cu at (122.2, 128.9)
- added TP39: TestPoint, PCM_7Sigma:TestPoint_Pad_D1.5mm, B.Cu at (126.4, 116.5)
- added TP40: TestPoint, PCM_7Sigma:TestPoint_Pad_D1.5mm, B.Cu at (129.3, 115.6)
- added TP42: TestPoint, PCM_7Sigma:TestPoint_Pad_D1.5mm, B.Cu at (120.0, 115.0)
- added TP43: TestPoint, PCM_7Sigma:TestPoint_Pad_D1.5mm, B.Cu at (117.7, 113.3)
- added TP44: TestPoint, PCM_7Sigma:TestPoint_Pad_D1.5mm, B.Cu at (131.4, 119.6)
- added TP45: TestPoint, PCM_7Sigma:TestPoint_Pad_D1.5mm, B.Cu at (121.5, 118.2)
- added TP46: TestPoint, PCM_7Sigma:TestPoint_Pad_D1.5mm, B.Cu at (118.1, 118.4)
- added TP47: TestPoint, PCM_7Sigma:TestPoint_Pad_D1.5mm, B.Cu at (134.3, 119.6)
- added TP48: TestPoint, PCM_7Sigma:TestPoint_Pad_D1.5mm, B.Cu at (134.0, 123.4)
- added TP49: TestPoint, PCM_7Sigma:TestPoint_Pad_D1.5mm, B.Cu at (131.6, 125.1)
- added TP50: TestPoint, PCM_7Sigma:TestPoint_Pad_D1.5mm, B.Cu at (154.7, 106.8)
- added TP51: TestPoint, PCM_7Sigma:TestPoint_Pad_D1.5mm, B.Cu at (147.4, 106.8)
- added TP52: TestPoint, PCM_7Sigma:TestPoint_Pad_D1.5mm, B.Cu at (142.2, 134.1)
- added TP53: TestPoint, PCM_7Sigma:TestPoint_Pad_D1.5mm, B.Cu at (142.0, 121.7)
- added TP7: TestPoint, PCM_7Sigma:TestPoint_Pad_D1.5mm, B.Cu at (138.3, 79.9)
- added TP8: TestPoint, PCM_7Sigma:TestPoint_Pad_D1.5mm, B.Cu at (139.0, 84.7)
- added TP9: TestPoint, PCM_7Sigma:TestPoint_Pad_D1.5mm, B.Cu at (143.3, 84.7)
- C1, C10, C11, C12, C13, C14, C15, C16, C17, C19, C20, C22, C24, C25, C26, C27, C28, C29, C30, C31, C32, C4, C40, C41, C46, C47, C48, C49, C50, C51, C52, C53, C54, C6, C62, C63, C64, C65, C66, C67, C68, C69, C7, C70, C71, C72, C8, C9, C90, C91: footprint 7Sigma:C_0402_1005Metric -> PCM_7Sigma:C_0402_1005Metric
- C2, C21, C23, C58, C85, C86, C87: footprint 7Sigma:C_0805_2012Metric -> PCM_7Sigma:C_0805_2012Metric
- C3, C42, C43, C44, C45, C5, C55, C56, C57, C78, C79: footprint 7Sigma:C_1210_3225Metric -> PCM_7Sigma:C_1210_3225Metric
- D1, D4, D5, D6: footprint 7Sigma:D_SOD-323 -> PCM_7Sigma:D_SOD-323
- D10, D11, D2, D3: footprint 7Sigma:LED_0402_1005Metric -> PCM_7Sigma:LED_0402_1005Metric
- D12, D13, D14: footprint 7Sigma:USON-10_2.5x1.0mm_P0.5mm -> PCM_7Sigma:USON-10_2.5x1.0mm_P0.5mm
- D7, D8, D9: footprint 7Sigma:D_SMA -> PCM_7Sigma:D_SMA
- ENC2: footprint 7Sigma:TAKACHI_SIM6-12-3W -> PCM_7Sigma:TAKACHI_SIM6-12-3W
- F1, F2, F3: footprint 7Sigma:Fuse_1206_3216Metric -> PCM_7Sigma:Fuse_1206_3216Metric
- FB1: footprint 7Sigma:L_0603_1608Metric -> PCM_7Sigma:L_0603_1608Metric
- G1: footprint 7Sigma:7Sigma_Logo -> PCM_7Sigma:7Sigma_Logo
- H1, H2, H3, H4: footprint 7Sigma:MountingHole_2.5mm_Pad_4mm -> PCM_7Sigma:MountingHole_2.5mm_Pad_4mm
- J1: footprint 7Sigma:USB-3.1-SMD_U262-161N-4BVC11 -> PCM_7Sigma:USB-3.1-SMD_U262-161N-4BVC11
- J11, J12: footprint 7Sigma:ANT-SMD_KH-IPEX-K501-29 -> PCM_7Sigma:ANT-SMD_KH-IPEX-K501-29
- J2, J3, J5, J6, J7: footprint 7Sigma:CONN-TH_XY302V-3.5-2P -> PCM_7Sigma:CONN-TH_XY302V-3.5-2P
- J4: footprint 7Sigma:RJ45-TH_RC01812 -> PCM_7Sigma:RJ45-TH_RC01812
- J9: footprint 7Sigma:SIM-SMD_NANO-SIM-TL6P-H1.35 -> PCM_7Sigma:SIM-SMD_NANO-SIM-TL6P-H1.35
- L1, L2: footprint 7Sigma:L_0402_1005Metric -> PCM_7Sigma:L_0402_1005Metric
- L4, L5: footprint 7Sigma:L_Changjiang_FTC404030S -> PCM_7Sigma:L_Changjiang_FTC404030S
- LP1, LP2, LP3: footprint 7Sigma:FIX-LEMB2-4.8V0-F -> PCM_7Sigma:FIX-LEMB2-4.8V0-F
- Q11, Q12, Q13, Q14, Q15, Q18, Q4, Q5, Q7, Q8: footprint 7Sigma:SOT-23-3 -> PCM_7Sigma:SOT-23-3
- Q3, Q6: footprint 7Sigma:DFN-8-1EP_3x3mm_P0.65mm_EP1.55x2.4mm -> PCM_7Sigma:DFN-8-1EP_3x3mm_P0.65mm_EP1.55x2.4mm
- R1, R10, R11, R12, R13, R14, R15, R16, R17, R18, R19, R2, R20, R21, R22, R23, R25, R26, R27, R28, R3, R30, R31, R33, R34, R35, R36, R4, R42, R43, R44, R45, R46, R47, R48, R49, R5, R51, R52, R55, R56, R57, R58, R59, R6, R60, R7, R71, R72, R8, R9: footprint 7Sigma:R_0402_1005Metric -> PCM_7Sigma:R_0402_1005Metric
- R50: footprint 7Sigma:R_0805_2012Metric -> PCM_7Sigma:R_0805_2012Metric
- SW1: footprint 7Sigma:SW-SMD_TS24CA -> PCM_7Sigma:SW-SMD_TS24CA
- SW2: footprint 7Sigma:SW-TH_4P-RA-L6.0-W6.0-H9.0 -> PCM_7Sigma:SW-TH_4P-RA-L6.0-W6.0-H9.0
- U1: footprint 7Sigma:VQFN-40-1EP_5x5mm_P0.4mm_EP3.3x3.3mm_ThermalVias -> PCM_7Sigma:VQFN-40-1EP_5x5mm_P0.4mm_EP3.3x3.3mm_ThermalVias
- U10, U7, U8, U9: footprint 7Sigma:UQFN-16_1.8x2.6mm_P0.4mm -> PCM_7Sigma:UQFN-16_1.8x2.6mm_P0.4mm
- U11: footprint 7Sigma:SOT-23-5 -> PCM_7Sigma:SOT-23-5
- U14, U4: footprint 7Sigma:SOT-23-6 -> PCM_7Sigma:SOT-23-6
- U15: footprint 7Sigma:VQFN-14_L3.5-W3.5-P0.50-BL-EP-ThermalVias -> PCM_7Sigma:VQFN-14_L3.5-W3.5-P0.50-BL-EP-ThermalVias
- U16: footprint 7Sigma:XCVR_LE910R1-EU -> PCM_7Sigma:XCVR_LE910R1-EU
- U17, U18, U20: footprint 7Sigma:LED-SMD_4P-L1.3-W1.3-P0.80_WS2812E-1313 -> PCM_7Sigma:LED-SMD_4P-L1.3-W1.3-P0.80_WS2812E-1313
- U2: footprint 7Sigma:SOIC-8_3.9x4.9mm_P1.27mm -> PCM_7Sigma:SOIC-8_3.9x4.9mm_P1.27mm
- U3: footprint 7Sigma:SOIC-8_5.3x5.3mm_P1.27mm -> PCM_7Sigma:SOIC-8_5.3x5.3mm_P1.27mm
- U5, U6: value PCF8574RGTR(UMW) -> PCF8574RGTR; footprint 7Sigma:QFN-16-1EP_3x3mm_P0.5mm_EP1.7x1.7mm_ThermalVias -> PCM_7Sigma:QFN-16-1EP_3x3mm_P0.5mm_EP1.7x1.7mm_ThermalVias
- Y1: footprint 7Sigma:Crystal_SMD_3225-4Pin_3.2x2.5mm -> PCM_7Sigma:Crystal_SMD_3225-4Pin_3.2x2.5mm
Connections:
- J4 pad SH: unconnected-(J4-PadSH) -> GND
Routing:
- net /MUX/IN_8: track 17.9 -> 44.0 mm, vias 2 -> 5
- net /MUX/IN_5: track 33.8 -> 39.4 mm
- net /MUX/IN_3: track 53.6 -> 48.1 mm
- net /MUX/IN_7: track 39.5 -> 44.7 mm
- net /MCU/O1_CTRL: track 90.0 -> 95.0 mm
- net 3V3: track 232.8 -> 237.7 mm, vias 30 -> 31
- net /MISC/VSUPPLY: track 112.4 -> 115.9 mm
- net /MUX/IN_2: track 49.2 -> 52.5 mm
- net /LTE/UART_TXD: track 38.5 -> 41.7 mm, vias 0 -> 1
- net /MUX/IN_1: track 51.2 -> 54.4 mm
- net /MUX/IN_6: track 36.6 -> 39.4 mm
- net /MCU/RST: track 99.0 -> 101.8 mm
- net /MCU/MODBUS_TX: track 38.8 -> 41.5 mm, vias 2 -> 3
- net Net-(U16B-C106/CTS): track 0.00 -> 2.51 mm, vias 0 -> 1
- net /MUX/OUT_B: track 101.1 -> 103.6 mm, vias 7 -> 8
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- added copper zone on B.Cu, net GND
