File: src/LE910R1.kicad_sch (KiCad schematic)
At the start: 26 parts, among them U16 LE910R1

Commit message: Layout progress
Parts:
- C48, C49, C54, C66: Price @1 USD (none) -> 0.0015; Price @100 USD (none) -> 0.0015; Price @Bulk USD (none) -> 0.0012; Price Bulk Qty (none) -> 1000; Price Source (none) -> LCSC; Price Updated (none) -> 2026-05-14
- C62, C63, C65, C67, C68, C69: Price @1 USD (none) -> 0.0012; Price @100 USD (none) -> 0.0012; Price @Bulk USD (none) -> 0.0009; Price Bulk Qty (none) -> 1000; Price Source (none) -> LCSC; Price Updated (none) -> 2026-05-14
- C64: Price @1 USD (none) -> 0.0308; Price @100 USD (none) -> 0.0308; Price @Bulk USD (none) -> 0.0209; Price Bulk Qty (none) -> 600; Price Source (none) -> LCSC; Price Updated (none) -> 2026-05-14
- C70, C71: Price @1 USD (none) -> 0.0238; Price @100 USD (none) -> 0.0238; Price @Bulk USD (none) -> 0.0190; Price Bulk Qty (none) -> 500; Price Source (none) -> LCSC; Price Updated (none) -> 2026-05-14; now not fitted
- C78, C79: Price @1 USD (none) -> 0.1071; Price @100 USD (none) -> 0.0850; Price @Bulk USD (none) -> 0.0636; Price Bulk Qty (none) -> 1000; Price Source (none) -> LCSC; Price Updated (none) -> 2026-05-14
- R46: Price @1 USD (none) -> 0.0008; Price @100 USD (none) -> 0.0008; Price @Bulk USD (none) -> 0.0006; Price Bulk Qty (none) -> 1000; Price Source (none) -> LCSC; Price Updated (none) -> 2026-05-14
- R51, R52: Price @1 USD (none) -> 0.0013; Price @100 USD (none) -> 0.0013; Price @Bulk USD (none) -> 0.0011; Price Bulk Qty (none) -> 1000; Price Source (none) -> LCSC; Price Updated (none) -> 2026-05-14
- U16: Price @Bulk USD (none) -> 7.0000; Price Source (none) -> Manual

Commit message: schematic cleanup, verification. GPIO9 pin pulldown changed to pullup.
Parts:
- removed C48, C49, C54, C66: 100nF, 7Sigma:C_0402_1005Metric, symbol Capacitor:CL05B104KO5NNNC
- removed C62, C63, C65, C67, C68, C69: 33pF, 7Sigma:C_0402_1005Metric, symbol Capacitor:CC0402JRNPO9BN330
- removed C64: 1uF, 7Sigma:C_0402_1005Metric, symbol Capacitor:GRM155R61H105KE05D
- removed C70, C71: 1.2pF, 7Sigma:C_0402_1005Metric, symbol Capacitor:GJM1555C1H1R2WB01D
- removed C78, C79: 47uF, 7Sigma:C_1210_3225Metric, symbol Capacitor:CS3225X7R476K160NRL
- removed R46: 0R, 7Sigma:R_0402_1005Metric, symbol Resistor:0402WGF0000TCE
- removed R51, R52: 10K, 7Sigma:R_0402_1005Metric, symbol Resistor:0402WGF1002TCE
- removed TP10, TP11, TP12, TP24, TP7, TP8, TP9: TestPoint, 7Sigma:TestPoint_Pad_D1.5mm, symbol TestPoints:TestPoint_Pad_D1.5mm
- removed U16: LE910R1, 7Sigma:XCVR_LE910R1-EU, symbol ICs:LE910R1-EU
Connections:
- no-connect marks 37 -> 0
Other:
- note removed: "MODULE INPUT"
- note removed: "MODULE OUTPUT"
- note removed: "PLACE CLOSE TO MODULE"
