File: src/LTE.kicad_sch (KiCad schematic)
At the start: 60 parts, among them J4 Conn_Coaxial, J9 SIM_NANO_Socket, Q18 SI2308A, Q7 BC817-40-7-F, Q8 BC817-40-7-F, U15 TXS0104ERGYR, U16 LE910R1

Commit message: final pcb that went to production
Parts:
- C44, C45, C55, C56, C57, C78, C79: symbol Capacitor:CS3225X7R476K160NRL -> Capacitor:CL32A476KOJNNNE; Dielectric X7R -> X5R; LCSC Part C5440143 -> C2932477; Manufacturer 1 Samwha Capacitor -> Samsung Electro-Mechanics; Manufacturer Part Number 1 CS3225X7R476K160NRL -> CL32A476KOJNNNE; Price @1 USD 0.1071 -> 0.2665; Price @100 USD 0.0850 -> 0.1851; Price @Bulk USD 0.0636 -> 0.1693; Price Updated 2026-05-14 -> 2026-06-14; Supplier Part Number 1 C5440143 -> C2932477
