File: src/LTE.kicad_sch (KiCad schematic)
At the start: 60 parts, among them J4 Conn_Coaxial, J9 SIM_NANO_Socket, Q18 SI2308A, Q7 BC817-40-7-F, Q8 BC817-40-7-F, U15 TXS0104ERGYR, U16 LE910R1

Commit message: Update PCB layout and schematics; add enclosure design files
Bump firmware submodule to WAN failover scenario-audit hardening +
zombie-LTE self-heal (round 2).

Co-Authored-By: Claude Sonnet 5 <noreply@anthropic.com>
Parts:
- removed J4: Conn_Coaxial, 7Sigma:SMA-SMD_BWSMA-KE-P001, symbol Connectors:BWSMA-KE-P001
- added C72: 100nF, 7Sigma:C_0402_1005Metric, symbol Capacitor:CL05B104KO5NNNC
- added J11: Conn_IPEX, 7Sigma:ANT-SMD_KH-IPEX-K501-29, symbol Connectors:KH-IPEX-K501-29
Connections:
- net GND: now also R51.2, R52.2, C72.2, J11.2 (Ext), J11.3 (Ext)
- net SIM_VCC: now also C72.1; no longer R51.2, R52.2
- net at C71.1, R46.2: now also J11.1 (In)
- no-connect marks 39 -> 40
