File: src/LTE.kicad_sch (KiCad schematic)
At the start: 61 parts, among them J11 Conn_IPEX, J9 SIM_NANO_Socket, Q18 SI2308A, Q7 BC817-40-7-F, Q8 BC817-40-7-F, U15 TXS0104ERGYR, U16 LE910R1

Commit message: pcb layout continued
Parts:
- C44, C45, C55, C56, C57, C78, C79: symbol Capacitor:CL32A476KOJNNNE -> Capacitor:CS3225X7R476K160NRL; Dielectric X5R -> X7R; LCSC Part C2932477 -> C5440143; Manufacturer 1 Samsung Electro-Mechanics -> Samwha Capacitor; Manufacturer Part Number 1 CL32A476KOJNNNE -> CS3225X7R476K160NRL; Price @1 USD 0.2665 -> 0.3615; Price @100 USD 0.1851 -> 0.2960; Price @Bulk USD 0.1693 -> 0.2339; Price Updated 2026-06-14 -> 2026-07-16; Supplier Part Number 1 C2932477 -> C5440143

Commit message: layout continued
Connections:
- net GND: now also J11.4 (PT)
- no-connect marks 40 -> 39
Other:
- moved on the sheet: C70, C71, J11, R46
