File: src/LTE.kicad_sch (KiCad schematic)
At the start: 61 parts, among them J11 Conn_IPEX, J9 SIM_NANO_Socket, Q18 SI2308A, Q7 BC817-40-7-F, Q8 BC817-40-7-F, U15 TXS0104ERGYR, U16 LE910R1

Commit message: layout + lib swap to http library. changed up the 10u and 47u caps for cheaper alternative
Parts:
- C44, C45, C55, C56, C57, C78, C79: footprint 7Sigma:C_1210_3225Metric -> PCM_7Sigma:C_1210_3225Metric; symbol Capacitor:CS3225X7R476K160NRL -> 7Sigma:CS3225X7R476K160NRL; Price @1 USD 0.3615 -> (none); Price @100 USD 0.2960 -> (none); Price @Bulk USD 0.2339 -> (none); Price Bulk Qty 1000 -> (none); Price Source LCSC -> (none); Price Updated 2026-07-16 -> (none)
- C48, C49, C50, C51, C54, C66, C72: footprint 7Sigma:C_0402_1005Metric -> PCM_7Sigma:C_0402_1005Metric; symbol Capacitor:CL05B104KO5NNNC -> 7Sigma:CL05B104KO5NNNC; Price @1 USD 0.0015 -> (none); Price @100 USD 0.0015 -> (none); Price @Bulk USD 0.0012 -> (none); Price Bulk Qty 1000 -> (none); Price Source LCSC -> (none); Price Updated 2026-05-14 -> (none)
- C52, C53: footprint 7Sigma:C_0402_1005Metric -> PCM_7Sigma:C_0402_1005Metric; symbol Capacitor:CL05B103KB5NNNC -> 7Sigma:CL05B103KB5NNNC; Price @1 USD 0.0016 -> (none); Price @100 USD 0.0016 -> (none); Price @Bulk USD 0.0013 -> (none); Price Bulk Qty 1000 -> (none); Price Source LCSC -> (none); Price Updated 2026-05-14 -> (none)
- C62, C63, C65, C67, C68, C69: footprint 7Sigma:C_0402_1005Metric -> PCM_7Sigma:C_0402_1005Metric; symbol Capacitor:CC0402JRNPO9BN330 -> 7Sigma:CC0402JRNPO9BN330; Manufacturer 1 YAGEO -> Yageo; Price @1 USD 0.0012 -> (none); Price @100 USD 0.0012 -> (none); Price @Bulk USD 0.0009 -> (none); Price Bulk Qty 1000 -> (none); Price Source LCSC -> (none); Price Updated 2026-05-14 -> (none)
- C64: footprint 7Sigma:C_0402_1005Metric -> PCM_7Sigma:C_0402_1005Metric; symbol Capacitor:GRM155R61H105KE05D -> 7Sigma:GRM155R61H105KE05D; Manufacturer 1 Murata Electronics -> Murata; Price @1 USD 0.0308 -> (none); Price @100 USD 0.0308 -> (none); Price @Bulk USD 0.0209 -> (none); Price Bulk Qty 600 -> (none); Price Source LCSC -> (none); Price Updated 2026-05-14 -> (none)
- C70, C71: footprint 7Sigma:C_0402_1005Metric -> PCM_7Sigma:C_0402_1005Metric; symbol Capacitor:GJM1555C1H1R2WB01D -> 7Sigma:GJM1555C1H1R2WB01D; Manufacturer 1 muRata -> Murata; Price @1 USD 0.0238 -> (none); Price @100 USD 0.0238 -> (none); Price @Bulk USD 0.0190 -> (none); Price Bulk Qty 500 -> (none); Price Source LCSC -> (none); Price Updated 2026-05-14 -> (none)
- D3: footprint 7Sigma:LED_0402_1005Metric -> PCM_7Sigma:LED_0402_1005Metric; symbol LEDs:LTST-C281KRKT -> 7Sigma:LTST-C281KRKT; Footprint_Name (none) -> 0402; Manufacturer 1 LITEON -> Lite-On; Price @1 USD 0.0396 -> (none); Price @100 USD 0.0396 -> (none); Price @Bulk USD 0.0266 -> (none); Price Bulk Qty 600 -> (none); Price Source LCSC -> (none); Price Updated 2026-05-14 -> (none)
- J11: footprint 7Sigma:ANT-SMD_KH-IPEX-K501-29 -> PCM_7Sigma:ANT-SMD_KH-IPEX-K501-29; symbol Connectors:KH-IPEX-K501-29 -> 7Sigma:KH-IPEX-K501-29; Manufacturer 1 kinghelm -> Kinghelm; Price @1 USD 0.0715 -> (none); Price @100 USD 0.0581 -> (none); Price @Bulk USD 0.0455 -> (none); Price Bulk Qty 1000 -> (none); Price Source LCSC -> (none); Price Updated 2026-07-16 -> (none)
- J9: footprint 7Sigma:SIM-SMD_NANO-SIM-TL6P-H1.35 -> PCM_7Sigma:SIM-SMD_NANO-SIM-TL6P-H1.35; symbol Connectors:NANO_SIM_TL6P_H1.35 -> 7Sigma:NANO_SIM_TL6P_H1.35; Manufacturer 1 SHOU HAN -> Shou Han; Price @1 USD 0.1994 -> (none); Price @100 USD 0.1579 -> (none); Price @Bulk USD 0.1180 -> (none); Price Bulk Qty 500 -> (none); Price Source LCSC -> (none); Price Updated 2026-05-14 -> (none)
- Q18: footprint 7Sigma:SOT-23-3 -> PCM_7Sigma:SOT-23-3; symbol Transistors:SI2308A -> 7Sigma:SI2308A; Manufacturer 1 UMW -> UMW (Youtai Semiconductor Co., Ltd.); Price @1 USD 0.0364 -> (none); Price @100 USD 0.0284 -> (none); Price @Bulk USD 0.0242 -> (none); Price Bulk Qty 300 -> (none); Price Source LCSC -> (none); Price Updated 2026-05-14 -> (none)
- Q7, Q8: footprint 7Sigma:SOT-23-3 -> PCM_7Sigma:SOT-23-3; symbol Transistors:BC817-40-7-F -> 7Sigma:BC817-40-7-F; Manufacturer 1 DIODES -> Diodes Incorporated; Price @1 USD 0.1029 -> (none); Price @100 USD 0.0828 -> (none); Price @Bulk USD 0.0653 -> (none); Price Bulk Qty 500 -> (none); Price Source LCSC -> (none); Price Updated 2026-05-14 -> (none)
- R20: footprint 7Sigma:R_0402_1005Metric -> PCM_7Sigma:R_0402_1005Metric; symbol Resistor:0402WGF1001TCE -> 7Sigma:0402WGF1001TCE; Manufacturer 1 Uni-Royal -> UNI-ROYAL(Uniroyal Elec); Price @1 USD 0.0011 -> (none); Price @100 USD 0.0011 -> (none); Price @Bulk USD 0.0009 -> (none); Price Bulk Qty 1000 -> (none); Price Source LCSC -> (none); Price Updated 2026-05-14 -> (none)
- R33, R34, R47: footprint 7Sigma:R_0402_1005Metric -> PCM_7Sigma:R_0402_1005Metric; symbol Resistor:0402WGF1003TCE -> 7Sigma:0402WGF1003TCE; Manufacturer 1 Uni-Royal -> UNI-ROYAL(Uniroyal Elec); Price @1 USD 0.0009 -> (none); Price @100 USD 0.0009 -> (none); Price @Bulk USD 0.0007 -> (none); Price Bulk Qty 1000 -> (none); Price Source LCSC -> (none); Price Updated 2026-05-14 -> (none)
- R35, R36, R45, R51, R52: footprint 7Sigma:R_0402_1005Metric -> PCM_7Sigma:R_0402_1005Metric; symbol Resistor:0402WGF1002TCE -> 7Sigma:0402WGF1002TCE; Manufacturer 1 Uni-Royal -> UNI-ROYAL(Uniroyal Elec); Price @1 USD 0.0013 -> (none); Price @100 USD 0.0013 -> (none); Price @Bulk USD 0.0011 -> (none); Price Bulk Qty 1000 -> (none); Price Source LCSC -> (none); Price Updated 2026-05-14 -> (none)
- R46: footprint 7Sigma:R_0402_1005Metric -> PCM_7Sigma:R_0402_1005Metric; symbol Resistor:0402WGF0000TCE -> 7Sigma:0402WGF0000TCE; Manufacturer 1 Uni-Royal -> UNI-ROYAL(Uniroyal Elec); Price @1 USD 0.0008 -> (none); Price @100 USD 0.0008 -> (none); Price @Bulk USD 0.0006 -> (none); Price Bulk Qty 1000 -> (none); Price Source LCSC -> (none); Price Updated 2026-05-14 -> (none)
- TP10, TP11, TP12, TP13, TP14, TP15, TP16, TP17, TP18, TP19, TP20, TP21, TP22, TP23, TP24, TP7, TP8, TP9: footprint 7Sigma:TestPoint_Pad_D1.5mm -> PCM_7Sigma:TestPoint_Pad_D1.5mm; symbol TestPoints:TestPoint_Pad_D1.5mm -> 7Sigma:TestPoint_Pad_D1.5mm
- U15: footprint 7Sigma:VQFN-14_L3.5-W3.5-P0.50-BL-EP-ThermalVias -> PCM_7Sigma:VQFN-14_L3.5-W3.5-P0.50-BL-EP-ThermalVias; symbol ICs:TXS0104ERGYR -> 7Sigma:TXS0104ERGYR; Bit Width (none) -> 4-Bit; Price @1 USD 0.3795 -> (none); Price @100 USD 0.2997 -> (none); Price @Bulk USD 0.1940 -> (none); Price Bulk Qty 500 -> (none); Price Source LCSC -> (none); Price Updated 2026-05-14 -> (none); VCCA Range (none) -> 1.65V–3.6V; VCCB Range (none) -> 2.3V–5.5V
- U16: footprint 7Sigma:XCVR_LE910R1-EU -> PCM_7Sigma:XCVR_LE910R1-EU; symbol ICs:LE910R1-EU -> 7Sigma:LE910R1-EU; Price @Bulk USD 7.0000 -> (none); Price Source Manual -> (none)
