File: src/MUX.kicad_sch (KiCad schematic)
At the start: 20 parts, among them U10 TMUX1208RSVR, U5 PCF8574RGTR(UMW), U6 PCF8574RGTR(UMW), U7 TMUX1208RSVR, U8 TMUX1208RSVR, U9 TMUX1208RSVR

Commit message: final pcb that went to production
Parts:
- C18, C33, C34, C35, C36, C37, C38, C39: symbol Capacitor:CC0402JRNPO9BN101 -> Capacitor:0402CG101J500NT; Dielectric NP0 -> C0G; LCSC Part C106200 -> C1546; Manufacturer 1 YAGEO -> FH; Manufacturer Part Number 1 CC0402JRNPO9BN101 -> 0402CG101J500NT; Price @1 USD 0.0012 -> 0.0020; Price @100 USD 0.0012 -> 0.0020; Price @Bulk USD 0.0010 -> 0.0017; Price Updated 2026-05-14 -> 2026-06-14; Supplier Part Number 1 C106200 -> C1546
