File: src/PWR.kicad_sch (KiCad schematic)
At the start: 59 parts, among them J1 USB_C_Receptacle_USB2.0_16P, Q1 AO3401A, Q11 SI2308A, Q12 SI2308A, Q13 SI2308A, Q2 AO3401A, U14 TPS54302DDCR, U19 TPS54302DDCR, U4 TPS54302DDCR

Commit message: final pcb that went to production
Parts:
- C20, C82: symbol Capacitor:CC0402JRNPO9BN101 -> Capacitor:0402CG101J500NT; Dielectric NP0 -> C0G; LCSC Part C106200 -> C1546; Manufacturer 1 YAGEO -> FH; Manufacturer Part Number 1 CC0402JRNPO9BN101 -> 0402CG101J500NT; Price @1 USD 0.0012 -> 0.0020; Price @100 USD 0.0012 -> 0.0020; Price @Bulk USD 0.0010 -> 0.0017; Price Updated 2026-05-14 -> 2026-06-14; Supplier Part Number 1 C106200 -> C1546
- C3, C42, C43, C5, C83, C93: symbol Capacitor:CS3225X7R476K160NRL -> Capacitor:CL32A476KOJNNNE; Dielectric X7R -> X5R; LCSC Part C5440143 -> C2932477; Manufacturer 1 Samwha Capacitor -> Samsung Electro-Mechanics; Manufacturer Part Number 1 CS3225X7R476K160NRL -> CL32A476KOJNNNE; Price @1 USD 0.1071 -> 0.2665; Price @100 USD 0.0850 -> 0.1851; Price @Bulk USD 0.0636 -> 0.1693; Price Updated 2026-05-14 -> 2026-06-14; Supplier Part Number 1 C5440143 -> C2932477
Other:
- note added: "10-28V secure against reverse polarity."
- note removed: "10-28V probably secure against reverse polarity."
- moved on the sheet: C21, C81, C82, C83, C87, C92, C93, D11, D12, L6, R37, R39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
