File: src/CE_Dongle_V3.kicad_sch (KiCad schematic)
At the start: 13 parts, among them J10 Conn_01x02, J2 Conn_01x02, J3 Conn_01x02, J6 Conn_01x02, J7 8P8C_LED_Shielded, J8 Conn_01x02

Commit message: Update PCB layout and schematics; add enclosure design files
Bump firmware submodule to WAN failover scenario-audit hardening +
zombie-LTE self-heal (round 2).

Co-Authored-By: Claude Sonnet 5 <noreply@anthropic.com>
Parts:
- removed ENC1: Hammond_1551XFLGY, 7Sigma:HAMMOND_1551XFLGY, symbol Mechanical_7S:Hammond_1551XFLGY
- removed J10, J2, J3, J6, J8: Conn_01x02, 7Sigma:CONN-TH_DB301V-3.5-2P-GN, symbol Connectors:DB301V-3.5-2P-GN-S
- removed J7: 8P8C_LED_Shielded, 7Sigma:RJ45-TH_RC01812, symbol Connectors:RC01812
- removed R29: 1K, 7Sigma:R_0402_1005Metric, symbol Resistor:0402WGF1001TCE
- added ENC2: Takachi_SIM6-12-3W, 7Sigma:TAKACHI_SIM6-12-3W, symbol Mechanical_7S:Takachi_SIM6-12-3W
- added J2, J3, J5, J6, J7: Conn_01x02, 7Sigma:CONN-TH_XY302V-3.5-2P, symbol Connectors:XY302V-3.5-2P
- added J4: 8P8C_LED_Shielded, 7Sigma:RJ45-TH_RC01812, symbol Connectors:RC01812
- added TP42, TP43, TP44, TP45, TP46, TP47, TP48, TP49: TestPoint, 7Sigma:TestPoint_Pad_D1.5mm, symbol TestPoints:TestPoint_Pad_D1.5mm
Connections:
- net GND: now also J3.1 (Pin_1), J5.2 (Pin_2), J6.1 (Pin_1)
- net MISC/TEMP_DATA: now also J2.2 (Pin_2)
- net MISC/TEMP_VCC: now also J2.1 (Pin_1)
- net MUX/IN_1: now also J4.1, TP46.1
- net MUX/IN_2: now also J4.2, TP47.1
- net MUX/IN_3: now also J4.3, TP48.1
- net MUX/IN_4: now also J4.4, TP49.1
- net MUX/IN_5: now also J4.5, TP45.1
- net MUX/IN_6: now also J4.6, TP44.1
- net MUX/IN_7: now also J4.7, TP43.1
- net MUX/IN_8: now also J4.8, TP42.1
- net MUX/OUT_A: now also J7.1 (Pin_1)
- net MUX/OUT_B: now also J7.2 (Pin_2)
- net PWR/V_EXT: now also J6.2 (Pin_2)
- new net MISC/OUT1: J3.2 (Pin_2)
- new net MISC/OUT2: J5.1 (Pin_1)
- no-connect marks 2 -> 0
Other:
- sheet MCU ports: added O1_CTRL, O2_CTRL; removed RY1_CTRL, RY2_CTRL
- sheet MISC ports: added O1_CTRL, O2_CTRL, OUT1, OUT2, V_SUP; removed R1_CTRL, R2_CTRL, RY1_COM, RY1_NO, RY2_COM, RY2_NO
- sheet PWR ports: added V_SUP; removed none
- note removed: "RY_COM"
