File: src/CE_Dongle_V3.kicad_sch (KiCad schematic)
At the start: 20 parts, among them J2 Conn_01x02, J3 Conn_01x02, J4 8P8C_LED_Shielded, J5 Conn_01x02, J6 Conn_01x02, J7 Conn_01x02

Commit message: layout + lib swap to http library. changed up the 10u and 47u caps for cheaper alternative
Parts:
- ENC2: footprint 7Sigma:TAKACHI_SIM6-12-3W -> PCM_7Sigma:TAKACHI_SIM6-12-3W; symbol Mechanical_7S:Takachi_SIM6-12-3W -> 7Sigma:Takachi_SIM6-12-3W; Datasheet 2 (none) -> http://localhost:8020/api/datasheets/292/file; Datasheet 3 (none) -> http://localhost:8020/api/datasheets/293/file; Manufacturer 1 Takachi -> TAKACHI
- G1: footprint 7Sigma:7Sigma_Logo -> PCM_7Sigma:7Sigma_Logo; symbol Mechanical_7S:7Sigma_Logo -> 7Sigma:7Sigma_Logo; now in the parts list
- H1, H2, H3, H4: footprint 7Sigma:MountingHole_2.5mm_Pad_4mm -> PCM_7Sigma:MountingHole_2.5mm_Pad_4mm; symbol Mechanical_7S:MH_2.5mm_4mm_OD -> 7Sigma:MH_2.5mm_4mm_OD; now in the parts list
- J2, J3, J5, J6, J7: footprint 7Sigma:CONN-TH_XY302V-3.5-2P -> PCM_7Sigma:CONN-TH_XY302V-3.5-2P; symbol Connectors:XY302V-3.5-2P -> 7Sigma:XY302V-3.5-2P; Manufacturer 1 XINLAIYA -> Xinlaiya; Price @1 USD 0.1532 -> (none); Price @100 USD 0.1204 -> (none); Price @Bulk USD 0.1064 -> (none); Price Bulk Qty 150 -> (none); Price Source LCSC -> (none); Price Updated 2026-07-19 -> (none)
- J4: footprint 7Sigma:RJ45-TH_RC01812 -> PCM_7Sigma:RJ45-TH_RC01812; symbol Connectors:RC01812 -> 7Sigma:RC01812; Price @1 USD 0.6010 -> (none); Price @100 USD 0.3363 -> (none); Price @Bulk USD 0.2908 -> (none); Price Bulk Qty 1000 -> (none); Price Source LCSC -> (none); Price Updated 2026-07-16 -> (none)
- TP42, TP43, TP44, TP45, TP46, TP47, TP48, TP49: footprint 7Sigma:TestPoint_Pad_D1.5mm -> PCM_7Sigma:TestPoint_Pad_D1.5mm; symbol TestPoints:TestPoint_Pad_D1.5mm -> 7Sigma:TestPoint_Pad_D1.5mm
Connections:
- net GND: now also J4.SH
