File: src/MCU.kicad_sch (KiCad schematic)
At the start: 44 parts, among them J5 Conn_Coaxial, SW1 TS24CA, SW2 KH-6X6X7H-STM, U1 ESP32-C6, U17 WS2812, U18 WS2812, U20 WS2812, U3 W25Q64JVSSIQ, Y1 40MHz

Commit message: Update PCB layout and schematics; add enclosure design files
Bump firmware submodule to WAN failover scenario-audit hardening +
zombie-LTE self-heal (round 2).

Co-Authored-By: Claude Sonnet 5 <noreply@anthropic.com>
Parts:
- removed J5: Conn_Coaxial, 7Sigma:SMA-SMD_BWSMA-KE-P001, symbol Connectors:BWSMA-KE-P001
- removed SW2: KH-6X6X7H-STM, 7Sigma:SW-SMD_4P-L6.0-W6.0-P4.50-LS9.0-H7.0, symbol Buttons:KH-6X6X7H-STM
- added J12: Conn_IPEX, 7Sigma:ANT-SMD_KH-IPEX-K501-29, symbol Connectors:KH-IPEX-K501-29
- added SW2: TC-6615-9.0-160G, 7Sigma:SW-TH_4P-RA-L6.0-W6.0-H9.0, symbol Buttons:TC-6615-9.0-160G
- added TP37, TP38, TP39, TP40, TP41: TestPoint, 7Sigma:TestPoint_Pad_D1.5mm, symbol TestPoints:TestPoint_Pad_D1.5mm
Connections:
- net BUTTON: now also SW2.3 (K), SW2.4 (A), TP38.1
- net GND: now also J12.2 (Ext), J12.3 (Ext), SW2.1, SW2.2
- net GPIO8: now also TP41.1
- net I2C_SCL: now also TP40.1
- net I2C_SDA: now also TP39.1
- net RST: now also TP37.1
- net at C15.1, L2.1: now also J12.1 (In)
- net RY1_CTRL renamed O1_CTRL
- net RY2_CTRL renamed O2_CTRL
- no-connect marks 6 -> 7
