File: src/MCU.kicad_sch (KiCad schematic)
At the start: 49 parts, among them J12 Conn_IPEX, SW1 TS24CA, SW2 TC-6615-9.0-160G, U1 ESP32-C6, U17 WS2812, U18 WS2812, U20 WS2812, U3 W25Q64JVSSIQ, Y1 40MHz

Commit message: layout continued
Connections:
- net GND: now also J12.4 (PT)
- no-connect marks 7 -> 6
Changed lines of the file:
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@@
+	)
+	(junction
+		(at 20.32 58.42)
+		(diameter 0)
+		(color 0 0 0 0)
 	)
 	(junction
@@
 	)
 	(no_connect
-		(at 17.78 53.34)
-	)
-	(no_connect
 		(at 99.06 45.72)
 	)
@@
 	(wire
 		(pts
+			(xy 17.78 58.42) (xy 20.32 58.42)
+		)
+		(stroke
+			(width 0)
+			(type default)
+		)
+	)
+	(wire
+		(pts
 			(xy 226.06 143.51) (xy 233.68 143.51)
 		)
@@
 		)
 		(stroke
+			(width 0)
+			(type default)
+		)
+	)
+	(wire
+		(pts
+			(xy 17.78 53.34) (xy 17.78 58.42)
+		)
+		(stroke
