File: src/MCU.kicad_sch (KiCad schematic)
At the start: 49 parts, among them J12 Conn_IPEX, SW1 TS24CA, SW2 TC-6615-9.0-160G, U1 ESP32-C6, U17 WS2812, U18 WS2812, U20 WS2812, U3 W25Q64JVSSIQ, Y1 40MHz

Commit message: layout + lib swap to http library. changed up the 10u and 47u caps for cheaper alternative
Parts:
- removed TP41: TestPoint, 7Sigma:TestPoint_Pad_D1.5mm, symbol TestPoints:TestPoint_Pad_D1.5mm
- C1, C4: footprint 7Sigma:C_0402_1005Metric -> PCM_7Sigma:C_0402_1005Metric; symbol Capacitor:GRM155R61H105KE05D -> 7Sigma:GRM155R61H105KE05D; Manufacturer 1 Murata Electronics -> Murata; Price @1 USD 0.0308 -> (none); Price @100 USD 0.0308 -> (none); Price @Bulk USD 0.0209 -> (none); Price Bulk Qty 600 -> (none); Price Source LCSC -> (none); Price Updated 2026-05-14 -> (none)
- C10, C11, C22, C25, C26, C46, C47, C7, C8, C9: footprint 7Sigma:C_0402_1005Metric -> PCM_7Sigma:C_0402_1005Metric; symbol Capacitor:CL05B104KO5NNNC -> 7Sigma:CL05B104KO5NNNC; Price @1 USD 0.0015 -> (none); Price @100 USD 0.0015 -> (none); Price @Bulk USD 0.0012 -> (none); Price Bulk Qty 1000 -> (none); Price Source LCSC -> (none); Price Updated 2026-05-14 -> (none)
- C12, C13: footprint 7Sigma:C_0402_1005Metric -> PCM_7Sigma:C_0402_1005Metric; symbol Capacitor:CL05A106MP5NUNC -> 7Sigma:CL05A106MP5NUNC; Manufacturer 1 Murata Electronics -> Murata; Price @1 USD 0.0090 -> (none); Price @100 USD 0.0090 -> (none); Price @Bulk USD 0.0064 -> (none); Price Bulk Qty 600 -> (none); Price Source LCSC -> (none); Price Updated 2026-05-14 -> (none)
- C14, C15: footprint 7Sigma:C_0402_1005Metric -> PCM_7Sigma:C_0402_1005Metric; symbol Capacitor:GJM1555C1H1R2WB01D -> 7Sigma:GJM1555C1H1R2WB01D; Manufacturer 1 muRata -> Murata; Price @1 USD 0.0238 -> (none); Price @100 USD 0.0238 -> (none); Price @Bulk USD 0.0190 -> (none); Price Bulk Qty 500 -> (none); Price Source LCSC -> (none); Price Updated 2026-05-14 -> (none)
- C16, C17: footprint 7Sigma:C_0402_1005Metric -> PCM_7Sigma:C_0402_1005Metric; symbol Capacitor:CC0402JRNPO9BN120 -> 7Sigma:CC0402JRNPO9BN120; Manufacturer 1 YAGEO -> Yageo; Price @1 USD 0.0012 -> (none); Price @100 USD 0.0012 -> (none); Price @Bulk USD 0.0009 -> (none); Price Bulk Qty 1000 -> (none); Price Source LCSC -> (none); Price Updated 2026-05-14 -> (none)
- J12: footprint 7Sigma:ANT-SMD_KH-IPEX-K501-29 -> PCM_7Sigma:ANT-SMD_KH-IPEX-K501-29; symbol Connectors:KH-IPEX-K501-29 -> 7Sigma:KH-IPEX-K501-29; Manufacturer 1 kinghelm -> Kinghelm; Price @1 USD 0.0715 -> (none); Price @100 USD 0.0581 -> (none); Price @Bulk USD 0.0455 -> (none); Price Bulk Qty 1000 -> (none); Price Source LCSC -> (none); Price Updated 2026-07-16 -> (none)
- L1, L2: footprint 7Sigma:L_0402_1005Metric -> PCM_7Sigma:L_0402_1005Metric; symbol Inductors:LQW15AN2N2C10D -> 7Sigma:LQW15AN2N2C10D; Manufacturer 1 muRata -> Murata Electronics; Price @1 USD 0.0490 -> (none); Price @100 USD 0.0402 -> (none); Price @Bulk USD 0.0324 -> (none); Price Bulk Qty 1000 -> (none); Price Source LCSC -> (none); Price Updated 2026-05-14 -> (none)
- LP1, LP2, LP3: footprint 7Sigma:FIX-LEMB2-4.8V0-F -> PCM_7Sigma:FIX-LEMB2-4.8V0-F; symbol Mechanical_7S:FIX-LEMB2-4.8V0-F -> 7Sigma:FIX-LEMB2-4.8V0-F; Head Diameter (none) -> 2.3mm; Length (none) -> 4.8mm; Mounting Hole Diameter (none) -> 1.98mm; Post Diameter (none) -> 1.9mm; Price @Bulk USD 0.0720 -> (none); Price Bulk Qty 1000 -> (none); Price Source Manual -> (none)
- R12, R13, R15, R16, R17: footprint 7Sigma:R_0402_1005Metric -> PCM_7Sigma:R_0402_1005Metric; symbol Resistor:0402WGF220JTCE -> 7Sigma:0402WGF220JTCE; Manufacturer 1 Uni-Royal -> UNI-ROYAL(Uniroyal Elec); Price @1 USD 0.0007 -> (none); Price @100 USD 0.0007 -> (none); Price @Bulk USD 0.0006 -> (none); Price Bulk Qty 1000 -> (none); Price Source LCSC -> (none); Price Updated 2026-05-14 -> (none)
- R14, R21, R22, R31: footprint 7Sigma:R_0402_1005Metric -> PCM_7Sigma:R_0402_1005Metric; symbol Resistor:0402WGF1002TCE -> 7Sigma:0402WGF1002TCE; Manufacturer 1 Uni-Royal -> UNI-ROYAL(Uniroyal Elec); Price @1 USD 0.0013 -> (none); Price @100 USD 0.0013 -> (none); Price @Bulk USD 0.0011 -> (none); Price Bulk Qty 1000 -> (none); Price Source LCSC -> (none); Price Updated 2026-05-14 -> (none)
- R18: footprint 7Sigma:R_0402_1005Metric -> PCM_7Sigma:R_0402_1005Metric; symbol Resistor:0402WGF1200TCE -> 7Sigma:0402WGF1200TCE; Manufacturer 1 Uni-Royal -> UNI-ROYAL(Uniroyal Elec); Price @1 USD 0.0011 -> (none); Price @100 USD 0.0011 -> (none); Price @Bulk USD 0.0009 -> (none); Price Bulk Qty 1000 -> (none); Price Source LCSC -> (none); Price Updated 2026-05-14 -> (none)
- R42, R43: footprint 7Sigma:R_0402_1005Metric -> PCM_7Sigma:R_0402_1005Metric; symbol Resistor:0402WGF5101TCE -> 7Sigma:0402WGF5101TCE; Manufacturer 1 Uni-Royal -> UNI-ROYAL(Uniroyal Elec); Price @1 USD 0.0009 -> (none); Price @100 USD 0.0009 -> (none); Price @Bulk USD 0.0007 -> (none); Price Bulk Qty 1000 -> (none); Price Source LCSC -> (none); Price Updated 2026-05-14 -> (none)
- SW1: footprint 7Sigma:SW-SMD_TS24CA -> PCM_7Sigma:SW-SMD_TS24CA; symbol Buttons:TS24CA -> 7Sigma:TS24CA; Manufacturer 1 SHOU HAN -> Shou Han; Price @1 USD 0.0252 -> (none); Price @100 USD 0.0252 -> (none); Price @Bulk USD 0.0171 -> (none); Price Bulk Qty 600 -> (none); Price Source LCSC -> (none); Price Updated 2026-05-14 -> (none)
- SW2: footprint 7Sigma:SW-TH_4P-RA-L6.0-W6.0-H9.0 -> PCM_7Sigma:SW-TH_4P-RA-L6.0-W6.0-H9.0; symbol Buttons:TC-6615-9.0-160G -> 7Sigma:TC-6615-9.0-160G; Price @1 USD 0.0365 -> (none); Price @100 USD 0.0365 -> (none); Price @Bulk USD 0.0243 -> (none); Price Bulk Qty 1000 -> (none); Price Source LCSC -> (none); Price Updated 2026-07-16 -> (none)
- TP37, TP38, TP39, TP40: footprint 7Sigma:TestPoint_Pad_D1.5mm -> PCM_7Sigma:TestPoint_Pad_D1.5mm; symbol TestPoints:TestPoint_Pad_D1.5mm -> 7Sigma:TestPoint_Pad_D1.5mm
- U1: footprint 7Sigma:VQFN-40-1EP_5x5mm_P0.4mm_EP3.3x3.3mm_ThermalVias -> PCM_7Sigma:VQFN-40-1EP_5x5mm_P0.4mm_EP3.3x3.3mm_ThermalVias; symbol ICs:ESP32-C6 -> 7Sigma:ESP32-C6; Manufacturer 1 Espressif -> Espressif Systems; Price @1 USD 2.7877 -> (none); Price @100 USD 2.1605 -> (none); Price @Bulk USD 2.0154 -> (none); Price Bulk Qty 1000 -> (none); Price Source LCSC -> (none); Price Updated 2026-05-14 -> (none)
- U17, U18, U20: footprint 7Sigma:LED-SMD_4P-L1.3-W1.3-P0.80_WS2812E-1313 -> PCM_7Sigma:LED-SMD_4P-L1.3-W1.3-P0.80_WS2812E-1313; symbol ICs:WS2812E-1313 -> 7Sigma:WS2812E-1313; Footprint_Name (none) -> SMD-4P 1.3x1.3mm; PWM Resolution (none) -> 8-bit; Price @1 USD 0.0817 -> (none); Price @100 USD 0.0639 -> (none); Price @Bulk USD 0.0484 -> (none); Price Bulk Qty 1000 -> (none); Price Source LCSC -> (none); Price Updated 2026-05-14 -> (none); Voltage Range (none) -> 3.7V~5.3V
- U3: footprint 7Sigma:SOIC-8_5.3x5.3mm_P1.27mm -> PCM_7Sigma:SOIC-8_5.3x5.3mm_P1.27mm; symbol ICs:W25Q64JVSSIQ -> 7Sigma:W25Q64JVSSIQ; Capacity (none) -> 64Mbit; Footprint_Name (none) -> SOIC-8 208mil; Manufacturer 1 Winbond Elec -> Winbond; Max Frequency (none) -> 133MHz; Price @1 USD 1.6443 -> (none); Price @100 USD 1.1886 -> (none); Price @Bulk USD 1.1156 -> (none); Price Bulk Qty 1000 -> (none); Price Source LCSC -> (none); Price Updated 2026-05-14 -> (none); Voltage Range (none) -> 2.7V~3.6V
- Y1: footprint 7Sigma:Crystal_SMD_3225-4Pin_3.2x2.5mm -> PCM_7Sigma:Crystal_SMD_3225-4Pin_3.2x2.5mm; symbol Timing_Components:XTM32040000FT00351001 -> 7Sigma:XTM32040000FT00351001; Footprint_Name (none) -> SMD3225-4P; Price @1 USD 0.0841 -> (none); Price @100 USD 0.0681 -> (none); Price @Bulk USD 0.0541 -> (none); Price Bulk Qty 500 -> (none); Price Source LCSC -> (none); Price Updated 2026-05-14 -> (none)
