File: src/Modbus.kicad_sch (KiCad schematic)
At the start: 7 parts, among them U2 SP3485

Commit message: Update PCB layout and schematics; add enclosure design files
Bump firmware submodule to WAN failover scenario-audit hardening +
zombie-LTE self-heal (round 2).

Co-Authored-By: Claude Sonnet 5 <noreply@anthropic.com>
Parts:
- added D14: 5.5V, 7Sigma:USON-10_2.5x1.0mm_P0.5mm, symbol Diodes:TPD4E05U06DQAR
- added TP25, TP26, TP27, TP28, TP29: TestPoint, 7Sigma:TestPoint_Pad_D1.5mm, symbol TestPoints:TestPoint_Pad_D1.5mm
Connections:
- net GND: now also D14.3 (GND), D14.8 (GND)
- net MODBUS_A: now also D14.1 (D1+), D14.10 (D1+), TP28.1
- net MODBUS_B: now also D14.5 (D2-), D14.6 (D2-), TP29.1
- net RX: now also TP26.1
- net TX: now also TP25.1
- net TX_EN: now also TP27.1
Other:
- moved on the sheet: R3
