File: src/Modbus.kicad_sch (KiCad schematic)
At the start: 13 parts, among them U2 SP3485

Commit message: layout + lib swap to http library. changed up the 10u and 47u caps for cheaper alternative
Parts:
- C6: footprint 7Sigma:C_0402_1005Metric -> PCM_7Sigma:C_0402_1005Metric; symbol Capacitor:CL05B104KO5NNNC -> 7Sigma:CL05B104KO5NNNC; Price @1 USD 0.0015 -> (none); Price @100 USD 0.0015 -> (none); Price @Bulk USD 0.0012 -> (none); Price Bulk Qty 1000 -> (none); Price Source LCSC -> (none); Price Updated 2026-05-14 -> (none)
- D14: footprint 7Sigma:USON-10_2.5x1.0mm_P0.5mm -> PCM_7Sigma:USON-10_2.5x1.0mm_P0.5mm; symbol Diodes:TPD4E05U06DQAR -> 7Sigma:TPD4E05U06DQAR; Footprint_Name (none) -> USON-10; Manufacturer Part Number 1 TPD4E05U06DQAR -> (none); Price @1 USD 0.0875 -> (none); Price @100 USD 0.0717 -> (none); Price @Bulk USD 0.0570 -> (none); Price Bulk Qty 500 -> (none); Price Source LCSC -> (none); Price Updated 2026-07-19 -> (none)
- D2: footprint 7Sigma:LED_0402_1005Metric -> PCM_7Sigma:LED_0402_1005Metric; symbol LEDs:LTST-C281KRKT -> 7Sigma:LTST-C281KRKT; Footprint_Name (none) -> 0402; Manufacturer 1 LITEON -> Lite-On; Price @1 USD 0.0396 -> (none); Price @100 USD 0.0396 -> (none); Price @Bulk USD 0.0266 -> (none); Price Bulk Qty 600 -> (none); Price Source LCSC -> (none); Price Updated 2026-05-14 -> (none)
- R1: footprint 7Sigma:R_0402_1005Metric -> PCM_7Sigma:R_0402_1005Metric; symbol Resistor:0402WGF1200TCE -> 7Sigma:0402WGF1200TCE; Manufacturer 1 Uni-Royal -> UNI-ROYAL(Uniroyal Elec); Price @1 USD 0.0011 -> (none); Price @100 USD 0.0011 -> (none); Price @Bulk USD 0.0009 -> (none); Price Bulk Qty 1000 -> (none); Price Source LCSC -> (none); Price Updated 2026-05-14 -> (none)
- R3, R4, R5: footprint 7Sigma:R_0402_1005Metric -> PCM_7Sigma:R_0402_1005Metric; symbol Resistor:0402WGF1001TCE -> 7Sigma:0402WGF1001TCE; Manufacturer 1 Uni-Royal -> UNI-ROYAL(Uniroyal Elec); Price @1 USD 0.0011 -> (none); Price @100 USD 0.0011 -> (none); Price @Bulk USD 0.0009 -> (none); Price Bulk Qty 1000 -> (none); Price Source LCSC -> (none); Price Updated 2026-05-14 -> (none)
- TP25, TP26, TP27, TP28, TP29: footprint 7Sigma:TestPoint_Pad_D1.5mm -> PCM_7Sigma:TestPoint_Pad_D1.5mm; symbol TestPoints:TestPoint_Pad_D1.5mm -> 7Sigma:TestPoint_Pad_D1.5mm
- U2: footprint 7Sigma:SOIC-8_3.9x4.9mm_P1.27mm -> PCM_7Sigma:SOIC-8_3.9x4.9mm_P1.27mm; symbol ICs:SP3485EN-L/TR -> 7Sigma:SP3485EN-L/TR; Price @1 USD 0.3077 -> (none); Price @100 USD 0.2063 -> (none); Price @Bulk USD 0.1685 -> (none); Price Bulk Qty 1000 -> (none); Price Source LCSC -> (none); Price Updated 2026-05-14 -> (none)
