File: src/MISC.kicad_sch (KiCad schematic)
At the start: 28 parts, among them Q14 SI2308A, Q15 SI2308A, Q3 AON7264E, Q6 AON7264E

Commit message: layout + lib swap to http library. changed up the 10u and 47u caps for cheaper alternative
Parts:
- C24: footprint 7Sigma:C_0402_1005Metric -> PCM_7Sigma:C_0402_1005Metric; symbol Capacitor:GRM155R61H105KE05D -> 7Sigma:GRM155R61H105KE05D; Manufacturer 1 Murata Electronics -> Murata; Price @1 USD 0.0308 -> (none); Price @100 USD 0.0308 -> (none); Price @Bulk USD 0.0209 -> (none); Price Bulk Qty 600 -> (none); Price Source LCSC -> (none); Price Updated 2026-05-14 -> (none)
- D1, D5: footprint 7Sigma:D_SOD-323 -> PCM_7Sigma:D_SOD-323; symbol Diodes:BZX384-C3V6,115 -> 7Sigma:BZX384-C3V6,115; Footprint_Name (none) -> SOD-323; Price @1 USD 0.0291 -> (none); Price @100 USD 0.0291 -> (none); Price @Bulk USD 0.0191 -> (none); Price Bulk Qty 600 -> (none); Price Source LCSC -> (none); Price Updated 2026-07-17 -> (none)
- D10, D11: footprint 7Sigma:LED_0402_1005Metric -> PCM_7Sigma:LED_0402_1005Metric; symbol LEDs:LTST-C281KRKT -> 7Sigma:LTST-C281KRKT; Footprint_Name (none) -> 0402; Manufacturer 1 LITEON -> Lite-On; Price @1 USD 0.0396 -> (none); Price @100 USD 0.0396 -> (none); Price @Bulk USD 0.0266 -> (none); Price Bulk Qty 600 -> (none); Price Source LCSC -> (none); Price Updated 2026-05-14 -> (none)
- D4, D6: footprint 7Sigma:D_SOD-323 -> PCM_7Sigma:D_SOD-323; symbol Diodes:BZX384-C12,115 -> 7Sigma:BZX384-C12,115; Footprint_Name (none) -> SOD-323; Price @1 USD 0.0296 -> (none); Price @100 USD 0.0296 -> (none); Price @Bulk USD 0.0195 -> (none); Price Bulk Qty 600 -> (none); Price Source LCSC -> (none); Price Updated 2026-07-17 -> (none)
- D7, D8: footprint 7Sigma:D_SMA -> PCM_7Sigma:D_SMA; symbol Diodes:SMAJ28A -> 7Sigma:SMAJ28A; Clamping Voltage (none) -> 45.4V; Footprint_Name (none) -> SMA; Price @1 USD 0.1321 -> (none); Price @100 USD 0.1099 -> (none); Price @Bulk USD 0.0904 -> (none); Price Bulk Qty 500 -> (none); Price Source LCSC -> (none); Price Updated 2026-07-17 -> (none)
- F1, F2: footprint 7Sigma:Fuse_1206_3216Metric -> PCM_7Sigma:Fuse_1206_3216Metric; symbol Circuit_Protection:BSMD1206-110-30V -> 7Sigma:BSMD1206-110-30V; Price @1 USD 0.1468 -> (none); Price @100 USD 0.1135 -> (none); Price @Bulk USD 0.0844 -> (none); Price Bulk Qty 500 -> (none); Price Source LCSC -> (none); Price Updated 2026-07-17 -> (none)
- Q14, Q15: footprint 7Sigma:SOT-23-3 -> PCM_7Sigma:SOT-23-3; symbol Transistors:SI2308A -> 7Sigma:SI2308A; Manufacturer 1 UMW -> UMW (Youtai Semiconductor Co., Ltd.); Price @1 USD 0.0364 -> (none); Price @100 USD 0.0284 -> (none); Price @Bulk USD 0.0242 -> (none); Price Bulk Qty 300 -> (none); Price Source LCSC -> (none); Price Updated 2026-05-14 -> (none)
- Q3, Q6: footprint 7Sigma:DFN-8-1EP_3x3mm_P0.65mm_EP1.55x2.4mm -> PCM_7Sigma:DFN-8-1EP_3x3mm_P0.65mm_EP1.55x2.4mm; symbol Transistors:AON7264E -> 7Sigma:AON7264E; Manufacturer 1 Alpha & Omega Semicon -> Alpha & Omega Semiconductor; Price @1 USD 0.2896 -> (none); Price @100 USD 0.2362 -> (none); Price @Bulk USD 0.1847 -> (none); Price Bulk Qty 500 -> (none); Price Source LCSC -> (none); Price Updated 2026-07-16 -> (none)
- R19, R23: footprint 7Sigma:R_0402_1005Metric -> PCM_7Sigma:R_0402_1005Metric; symbol Resistor:0402WGF1001TCE -> 7Sigma:0402WGF1001TCE; Manufacturer 1 Uni-Royal -> UNI-ROYAL(Uniroyal Elec); Price @1 USD 0.0011 -> (none); Price @100 USD 0.0011 -> (none); Price @Bulk USD 0.0009 -> (none); Price Bulk Qty 1000 -> (none); Price Source LCSC -> (none); Price Updated 2026-05-14 -> (none)
- R44: footprint 7Sigma:R_0402_1005Metric -> PCM_7Sigma:R_0402_1005Metric; symbol Resistor:0402WGF1200TCE -> 7Sigma:0402WGF1200TCE; Manufacturer 1 Uni-Royal -> UNI-ROYAL(Uniroyal Elec); Price @1 USD 0.0011 -> (none); Price @100 USD 0.0011 -> (none); Price @Bulk USD 0.0009 -> (none); Price Bulk Qty 1000 -> (none); Price Source LCSC -> (none); Price Updated 2026-05-14 -> (none)
- R49: footprint 7Sigma:R_0402_1005Metric -> PCM_7Sigma:R_0402_1005Metric; symbol Resistor:0402WGF5101TCE -> 7Sigma:0402WGF5101TCE; Manufacturer 1 Uni-Royal -> UNI-ROYAL(Uniroyal Elec); Price @1 USD 0.0009 -> (none); Price @100 USD 0.0009 -> (none); Price @Bulk USD 0.0007 -> (none); Price Bulk Qty 1000 -> (none); Price Source LCSC -> (none); Price Updated 2026-05-14 -> (none)
- R50: footprint 7Sigma:R_0805_2012Metric -> PCM_7Sigma:R_0805_2012Metric; symbol Resistor:0805W8F1200T5E -> 7Sigma:0805W8F1200T5E; Manufacturer 1 Uni-Royal -> UNI-ROYAL(Uniroyal Elec); Price @1 USD 0.0028 -> (none); Price @100 USD 0.0028 -> (none); Price @Bulk USD 0.0022 -> (none); Price Bulk Qty 1000 -> (none); Price Source LCSC -> (none); Price Updated 2026-05-14 -> (none)
- R57, R58, R59, R60: footprint 7Sigma:R_0402_1005Metric -> PCM_7Sigma:R_0402_1005Metric; symbol Resistor:0402WGF2202TCE -> 7Sigma:0402WGF2202TCE; Manufacturer 1 Uni-Royal -> UNI-ROYAL(Uniroyal Elec); Price @1 USD 0.0010 -> (none); Price @100 USD 0.0010 -> (none); Price @Bulk USD 0.0008 -> (none); Price Bulk Qty 1000 -> (none); Price Source LCSC -> (none); Price Updated 2026-05-14 -> (none)
- TP50, TP51, TP52, TP53: footprint 7Sigma:TestPoint_Pad_D1.5mm -> PCM_7Sigma:TestPoint_Pad_D1.5mm; symbol TestPoints:TestPoint_Pad_D1.5mm -> 7Sigma:TestPoint_Pad_D1.5mm
